Commit message: [URDF]modified urdf model for new male mechanism

File: robots/assemble_quadrotors/urdf/assemble_dual_quadrotors_male.urdf.xacro (robot description, xacro)
@@ -17,5 +17,5 @@
   <!-- <xacro:property name="opt_pich_4" value="${0.348489}" /> -->
   <!-- <xacro:property name="opt_yaw_4" value="${-0.673131}" /> -->
-    <xacro:property name="pos_bound" value="${0.22628}" />
+  <xacro:property name="pos_bound" value="${0.22628}" />
   <xacro:property name="center_dis" value="${0.393}" />
   <xacro:property name="rotor_z" value="${0.052}" />
@@ -68,5 +68,5 @@
       <inertial>
         <origin xyz="0 0 0" rpy="0 0 0"/>
-        <mass value="0.0091"/>
+        <mass value="0.0000"/>
         <inertia
             ixx="0.00000807" ixy="0.0" ixz="0.0"
@@ -120,15 +120,15 @@
   <link name="main_body">
     <inertial>
-      <mass value = "0.78550624" />
+      <mass value = "1.01367590" />
       <origin xyz="0 0 0" rpy="0 0 0"/>
     <inertia
-        ixx="0.005554124" ixy="0.00002714" ixz="-0.00046661"
-        iyy="0.00758289" iyz="-0.00001400"
-        izz="0.011148881"/>
+        ixx="0.00642994" ixy="0.00003030" ixz="-0.00081536"
+        iyy="0.00964036" iyz="-0.00002604"
+        izz="0.01352704"/>
     </inertial>
     <visual>
       <origin rpy="0 0 0" xyz="0 0 0"/>
       <geometry>
-        <mesh filename="package://assemble_quadrotors/urdf/mesh/Assemble_dual_quadrotors_v3_male.STL"/>
+        <mesh filename="package://assemble_quadrotors/urdf/mesh/Assemble_quadrotor_male_v5.STL"/>
       </geometry>
     </visual>

Commit message: [URDF] modification for the inertia of male unit

File: robots/assemble_quadrotors/urdf/assemble_dual_quadrotors_male.urdf.xacro (robot description, xacro)
@@ -121,5 +121,5 @@
     <inertial>
       <mass value = "1.01367590" />
-      <origin xyz="0 0 0" rpy="0 0 0"/>
+      <origin xyz="0.02 0.0 0.02" rpy="0 0 0"/>
     <inertia
         ixx="0.00642994" ixy="0.00003030" ixz="-0.00081536"

Commit message: [URDF] modification about inertial information of male and neutral

File: robots/assemble_quadrotors/urdf/assemble_dual_quadrotors_male.urdf.xacro (robot description, xacro)
@@ -68,5 +68,5 @@
       <inertial>
         <origin xyz="0 0 0" rpy="0 0 0"/>
-        <mass value="0.0000"/>
+        <mass value="0.0052"/>
         <inertia
             ixx="0.00000807" ixy="0.0" ixz="0.0"
@@ -120,10 +120,10 @@
   <link name="main_body">
     <inertial>
-      <mass value = "1.01367590" />
-      <origin xyz="0.02 0.0 0.02" rpy="0 0 0"/>
+      <mass value = "0.99287590" />
+      <origin xyz="0.0209037 -0.00157892 0.00576541" rpy="0 0 0"/>
     <inertia
-        ixx="0.00642994" ixy="0.00003030" ixz="-0.00081536"
-        iyy="0.00964036" iyz="-0.00002604"
-        izz="0.01352704"/>
+        ixx="0.00608728" ixy="0.00003070" ixz="-0.00079536"
+        iyy="0.00932989" iyz="-0.00002784"
+        izz="0.01298518"/>
     </inertial>
     <visual>

File: robots/assemble_quadrotors/urdf/assemble_dual_quadrotors_neutral.urdf.xacro (robot description, xacro)
@@ -9,12 +9,4 @@
   <xacro:property name="center_dis" value="${0.393}" />
   <xacro:property name="rotor_z" value="${0.050}" />
-  <!-- <xacro:property name="opt_pich_1" value="${0.523525}" /> -->
-  <!-- <xacro:property name="opt_yaw_1" value="${0.73108}" /> -->
-  <!-- <xacro:property name="opt_pich_2" value="${0.523535}" /> -->
-  <!-- <xacro:property name="opt_yaw_2" value="${-2.08113}" /> -->
-  <!-- <xacro:property name="opt_pich_3" value="${0.523595}" /> -->
-  <!-- <xacro:property name="opt_yaw_3" value="${2.4662}" /> -->
-  <!-- <xacro:property name="opt_pich_4" value="${0.348489}" /> -->
-  <!-- <xacro:property name="opt_yaw_4" value="${-0.673131}" /> -->
   <xacro:property name="opt_pich_1" value="${0.45}" />
   <xacro:property name="opt_yaw_1" value="${0.73108}" />
@@ -117,10 +109,10 @@
   <link name="main_body">
     <inertial>
-      <mass value = "0.65877839" />
-      <origin xyz="0 0 0 " rpy="0 0 0"/>
+      <mass value = "0.83259112" />
+      <origin xyz="-0.00177281 0 0.017 " rpy="0 0 0"/>
       <inertia
-          ixx="0.00511034" ixy="-0.00012535" ixz="-0.00002267"
-          iyy="0.00537974" iyz="-0.00003189"
-          izz="0.00921821"/>
+          ixx="0.00572241" ixy="-0.00001571" ixz="0.00008325"
+          iyy="0.00609609" iyz="-0.00001479"
+          izz="0.01007121"/>
     </inertial>
     <visual>

Commit message: [URDF] corrected male urdf

File: robots/assemble_quadrotors/urdf/assemble_dual_quadrotors_male.urdf.xacro (robot description, xacro)
@@ -119,5 +119,5 @@
       <origin rpy="0 0 0" xyz="0 0 0"/>
       <geometry>
-        <mesh filename="package://assemble_quadrotors/urdf/mesh/Assemble_quadrotor_male_v5.STL"/>
+        <mesh filename="package://assemble_quadrotors/urdf/mesh/Assemble_dual_quadrotors_male_v4.STL"/>
       </geometry>
     </visual>
