Commit message: modified nuetral model with vim4

File: robots/assemble_quadrotors/urdf/assemble_dual_quadrotors_neutral.urdf.xacro (robot description, xacro)
@@ -118,14 +118,14 @@
     <inertial>
       <mass value = "0.65877839" />
-      <origin xyz="0 0 0 " rpy="0 0 0"/>
+      <origin xyz="0.00604808 0.00638317 0.01060495 " rpy="0 0 0"/>
       <inertia
-          ixx="0.00511034" ixy="-0.00012535" ixz="-0.00002267"
-          iyy="0.00537974" iyz="-0.00003189"
-          izz="0.00921821"/>
+          ixx="0.00605053" ixy="-0.00001519" ixz="0.00008891"
+          iyy="0.00638250" iyz="-0.00001297"
+          izz="0.01060318"/>
     </inertial>
     <visual>
       <origin rpy="0 0 0" xyz="0 0 0"/>
       <geometry>
-        <mesh filename="package://assemble_quadrotors/urdf/mesh/Assemble_dual_quadrotors_v3_neutral.STL" />
+        <mesh filename="package://assemble_quadrotors/urdf/mesh/Assemble_dual_quadrotors_v4_neutral.STL" />
       </geometry>
     </visual>
@@ -142,5 +142,5 @@
     <inertial>
       <mass value = "0.05" />
-      <origin xyz="0 0 0" rpy="0 0 0"/>
+      <origin xyz="-0.01 0 0" rpy="0 0 0"/>
       <inertia
           ixx="0.00001" ixy="0.0" ixz="0.0"

Commit message: [URDF] add new neutral model

File: robots/assemble_quadrotors/urdf/assemble_dual_quadrotors_neutral.urdf.xacro (robot description, xacro)
@@ -119,5 +119,5 @@
       <origin rpy="0 0 0" xyz="0 0 0"/>
       <geometry>
-        <mesh filename="package://assemble_quadrotors/urdf/mesh/Assemble_dual_quadrotors_v3_neutral.STL" />
+        <mesh filename="package://assemble_quadrotors/urdf/mesh/Assemble_dual_quadrotors_v4_neutral.STL" />
       </geometry>
     </visual>
