Commit message: [URDF] corrected imu origin

File: robots/assemble_quadrotors/urdf/assemble_dual_quadrotors_whole_female.urdf.xacro (robot description, xacro)
@@ -110,5 +110,6 @@
     <inertial>
       <mass value = "2.114" />
-      <origin xyz="0.00401288 0.00002524 0.00751852" rpy="0 0 0"/>
+      <!-- <origin xyz="0.00401288 0.00002524 0.00751852" rpy="0 0 0"/> -->
+      <origin xyz="0.0 0.0 0.0" rpy="0 0 0"/>
       <inertia
           ixx="0.01198006" ixy="0.00062162" ixz="-0.00032982"
@@ -131,5 +132,5 @@
   <!-- spinal -->
   <xacro:extra_module name = "fc" parent = "main_body" visible = "0" >
-    <origin xyz="-0.2 0.0 0.0165" rpy="0 0 0"/>
+    <origin xyz="-0.22 0.0 0.0165" rpy="0 0 0"/>
     <inertial>
       <mass value = "0.05" />

File: robots/assemble_quadrotors/urdf/assemble_dual_quadrotors_whole_male.urdf.xacro (robot description, xacro)
@@ -110,5 +110,6 @@
     <inertial>
       <mass value = "2.114" />
-      <origin xyz="-0.00401288 0.00002524 0.00751852" rpy="0 0 0"/>
+      <!-- <origin xyz="-0.00401288 0.00002524 0.00751852" rpy="0 0 0"/> -->
+      <origin xyz="0.0 0.00 0.00" rpy="0 0 0"/>
       <inertia
           ixx="0.01198006" ixy="0.00062162" ixz="0.00027258"
@@ -131,5 +132,5 @@
   <!-- spinal -->
   <xacro:extra_module name = "fc" parent = "main_body" visible = "0" >
-    <origin xyz="-0.2 0.0 0.0165" rpy="0 0 0"/>
+    <origin xyz="-0.22 0.0 0.0165" rpy="0 0 0"/>
     <inertial>
       <mass value = "0.05" />

Commit message: [URDF] corrected whole airframe origin

File: robots/assemble_quadrotors/urdf/assemble_dual_quadrotors_whole_female.urdf.xacro (robot description, xacro)
@@ -111,5 +111,6 @@
       <mass value = "2.114" />
       <!-- <origin xyz="0.00401288 0.00002524 0.00751852" rpy="0 0 0"/> -->
-      <origin xyz="0.0 0.0 0.0" rpy="0 0 0"/>
+      <origin xyz="0.00401288 0.0002524 0.00751852" rpy="0 0 0"/> <!-- for wired -->
+      <!-- <origin xyz="0.0 0.0 0.0" rpy="0 0 0"/> -->
       <inertia
           ixx="0.01198006" ixy="0.00062162" ixz="-0.00032982"

File: robots/assemble_quadrotors/urdf/assemble_dual_quadrotors_whole_male.urdf.xacro (robot description, xacro)
@@ -111,5 +111,6 @@
       <mass value = "2.114" />
       <!-- <origin xyz="-0.00401288 0.00002524 0.00751852" rpy="0 0 0"/> -->
-      <origin xyz="0.0 0.00 0.00" rpy="0 0 0"/>
+      <origin xyz="-0.00401288 -0.0002524 0.00751852" rpy="0 0 0"/> <!-- for wierd -->
+      <!-- <origin xyz="0.0 0.00 0.00" rpy="0 0 0"/> -->
       <inertia
           ixx="0.01198006" ixy="0.00062162" ixz="0.00027258"

Commit message: [URDF]modified whole robot models

File: robots/assemble_quadrotors/urdf/assemble_dual_quadrotors_whole_female.urdf.xacro (robot description, xacro)
@@ -109,12 +109,12 @@
   <link name="main_body">
     <inertial>
-      <mass value = "2.114" />
+      <mass value = "2.318" />
       <!-- <origin xyz="0.00401288 0.00002524 0.00751852" rpy="0 0 0"/> -->
-      <origin xyz="0.00401288 0.0002524 0.00751852" rpy="0 0 0"/> <!-- for wired -->
+      <origin xyz="0.00363315 -0.00001636 0.00477654" rpy="0 0 0"/> <!-- for wierd -->
       <!-- <origin xyz="0.0 0.0 0.0" rpy="0 0 0"/> -->
       <inertia
-          ixx="0.01198006" ixy="0.00062162" ixz="-0.00032982"
-          iyy="0.08096541" iyz="0.00000195"
-          izz="0.08846491"/>
+          ixx="0.01231937" ixy="0.00082883" ixz="-0.00028830"
+          iyy="0.11563003" iyz="0.00000115"
+          izz="0.12314029"/>
     </inertial>
     <visual>

File: robots/assemble_quadrotors/urdf/assemble_dual_quadrotors_whole_male.urdf.xacro (robot description, xacro)
@@ -109,12 +109,12 @@
   <link name="main_body">
     <inertial>
-      <mass value = "2.114" />
+      <mass value = "2.318" />
       <!-- <origin xyz="-0.00401288 0.00002524 0.00751852" rpy="0 0 0"/> -->
-      <origin xyz="-0.00401288 -0.0002524 0.00751852" rpy="0 0 0"/> <!-- for wierd -->
+      <origin xyz="-0.00363315 0.00001636 0.00477654" rpy="0 0 0"/> <!-- for wierd -->
       <!-- <origin xyz="0.0 0.00 0.00" rpy="0 0 0"/> -->
       <inertia
-          ixx="0.01198006" ixy="0.00062162" ixz="0.00027258"
-          iyy="0.08096541" iyz="-0.00000195"
-          izz="0.08846491"/>
+          ixx="0.01231937" ixy="0.00082883" ixz="0.00028830"
+          iyy="0.11563003" iyz="-0.00000115"
+          izz="0.12314029"/>
     </inertial>
     <visual>
