Commit message: work for the tuning of realmachines

File: robots/assemble_quadrotors/urdf/assemble_dual_quadrotors_female.urdf.xacro (robot description, xacro)
@@ -8,13 +8,13 @@
   <xacro:property name="pos_bound" value="${0.22628}" />
   <xacro:property name="center_dis" value="${0.393}" />
-  <xacro:property name="rotor_z" value="${0.050}" />
-  <xacro:property name="opt_pich_1" value="${0.523525}" />
+  <xacro:property name="rotor_z" value="${0.052}" />
+  <xacro:property name="opt_pich_1" value="${0.45}" />
   <xacro:property name="opt_yaw_1" value="${0.73108}" />
   <xacro:property name="opt_pich_2" value="${0.523535}" />
   <xacro:property name="opt_yaw_2" value="${-2.08113}" />
-  <xacro:property name="opt_pich_3" value="${0.523595}" />
-  <xacro:property name="opt_yaw_3" value="${2.4662}" />
-  <xacro:property name="opt_pich_4" value="${0.348489}" />
-  <xacro:property name="opt_yaw_4" value="${-0.673131}" />
+  <xacro:property name="opt_pich_3" value="${0.523535}" />
+  <xacro:property name="opt_yaw_3" value="${2.08113}" />
+  <xacro:property name="opt_pich_4" value="${0.45}" />
+  <xacro:property name="opt_yaw_4" value="${-0.73108}" />
   <!-- dynamics -->
   <m_f_rate value="-0.006" /> <!-- drag torque rate, the true value should be -0.006 -->
@@ -112,7 +112,7 @@
       <origin xyz="0 0 0 " rpy="0 0 0"/>
       <inertia
-          ixx="0.00558137" ixy="-0.00014117" ixz="-0.00047401"
-          iyy="0.00776130" iyz="0.00003630"
-          izz="0.01172792"/>
+          ixx="0.00523481" ixy="-0.00011631" ixz="-0.00040281"
+          iyy="0.00740303" iyz="-0.00003402"
+          izz="0.01114830"/>
     </inertial>
     <visual>
@@ -142,7 +142,7 @@
   </xacro:extra_module>
   <!-- propellers -->
-  <xacro:propeller_module id = "1" x = "-0.1044" y = "-0.12014" z = "0.05402" pich = "${opt_pich_4}" yaw = "${opt_yaw_4}" direction = "1" />
-  <xacro:propeller_module id = "2" x = "0.10705" y = "-0.10827" z = "0.05946" pich = "${opt_pich_3}" yaw = "${opt_yaw_3}"  direction = "-1" />
-  <xacro:propeller_module id = "3" x = "0.10474" y = "0.10579" z = "0.05404"  pich = "${opt_pich_2}" yaw = "${opt_yaw_2}" direction = "1" />
-  <xacro:propeller_module id = "4" x = "-0.10757" y = "0.12281" z = "0.05404"  pich = "${opt_pich_1}" yaw = "${opt_yaw_1}"  direction = "-1" />
+  <xacro:propeller_module id = "1" x = "-0.1044" y = "-0.12014" z = "0.05402" pich = "${-opt_pich_3}" yaw = "${opt_yaw_3}" direction = "1" />
+  <xacro:propeller_module id = "2" x = "0.10705" y = "-0.10827" z = "0.05946" pich = "${-opt_pich_4}" yaw = "${opt_yaw_4}"  direction = "-1" />
+  <xacro:propeller_module id = "3" x = "0.10705" y = "0.10827" z = "0.05402"  pich = "${-opt_pich_1}" yaw = "${opt_yaw_1}" direction = "1" />
+  <xacro:propeller_module id = "4" x = "-0.10705" y = "0.12014" z = "0.05404"  pich = "${-opt_pich_2}" yaw = "${opt_yaw_2}"  direction = "-1" />
 </robot>

File: robots/assemble_quadrotors/urdf/assemble_dual_quadrotors_male.urdf.xacro (robot description, xacro)
@@ -6,15 +6,26 @@
   <thrust_link name="thrust" />
   <!-- kinematics [m] -->
-  <xacro:property name="pos_bound" value="${0.22628}" />
+  <!-- <xacro:property name="pos_bound" value="${0.22628}" /> -->
+  <!-- <xacro:property name="center_dis" value="${0.393}" /> -->
+  <!-- <xacro:property name="rotor_z" value="${0.05}" /> -->
+  <!-- <xacro:property name="opt_pich_1" value="${0.523525}" /> -->
+  <!-- <xacro:property name="opt_yaw_1" value="${0.73108}" /> -->
+  <!-- <xacro:property name="opt_pich_2" value="${0.523535}" /> -->
+  <!-- <xacro:property name="opt_yaw_2" value="${-2.08113}" /> -->
+  <!-- <xacro:property name="opt_pich_3" value="${0.523595}" /> -->
+  <!-- <xacro:property name="opt_yaw_3" value="${2.4662}" /> -->
+  <!-- <xacro:property name="opt_pich_4" value="${0.348489}" /> -->
+  <!-- <xacro:property name="opt_yaw_4" value="${-0.673131}" /> -->
+    <xacro:property name="pos_bound" value="${0.22628}" />
   <xacro:property name="center_dis" value="${0.393}" />
-  <xacro:property name="rotor_z" value="${0.05}" />
-  <xacro:property name="opt_pich_1" value="${0.523525}" />
+  <xacro:property name="rotor_z" value="${0.052}" />
+  <xacro:property name="opt_pich_1" value="${0.45}" />
   <xacro:property name="opt_yaw_1" value="${0.73108}" />
   <xacro:property name="opt_pich_2" value="${0.523535}" />
   <xacro:property name="opt_yaw_2" value="${-2.08113}" />
-  <xacro:property name="opt_pich_3" value="${0.523595}" />
-  <xacro:property name="opt_yaw_3" value="${2.4662}" />
-  <xacro:property name="opt_pich_4" value="${0.348489}" />
-  <xacro:property name="opt_yaw_4" value="${-0.673131}" />
+  <xacro:property name="opt_pich_3" value="${0.523535}" />
+  <xacro:property name="opt_yaw_3" value="${2.08113}" />
+  <xacro:property name="opt_pich_4" value="${0.45}" />
+  <xacro:property name="opt_yaw_4" value="${-0.73108}" />
   <!-- dynamics -->
   <m_f_rate value="-0.006" /> <!-- drag torque rate, the true value should be -0.006 -->
@@ -112,8 +123,14 @@
       <mass value = "0.79154967" />
       <origin xyz="0 0 0" rpy="0 0 0"/>
-      <inertia
-          ixx="0.00565753" ixy="-0.00012094" ixz="0.00049859"
-          iyy="0.00763738" iyz="0.00003798"
-          izz="0.01152518"/>
+    <!--   <inertia -->
+    <!--       ixx="0.00565753" ixy="-0.00012094" ixz="0.00049859" -->
+    <!--       iyy="0.00763738" iyz="0.00003798" -->
+    <!--       izz="0.01152518"/> -->
+    <!-- </inertial> -->
+    <!--TODO modify to the correct inertia -->
+    <inertia
+        ixx="0.00523481" ixy="-0.00011631" ixz="-0.00040281"
+        iyy="0.00740303" iyz="-0.00003402"
+        izz="0.01114830"/>
     </inertial>
     <visual>
@@ -143,7 +160,11 @@
   </xacro:extra_module>
   <!-- propellers -->
-  <xacro:propeller_module id = "1" x = "${-pos_bound/2}" y = "${-pos_bound/2}" z = "${rotor_z}" pich = "${opt_pich_1}" yaw = "${opt_yaw_1}" direction = "1" />
-  <xacro:propeller_module id = "2" x = "${pos_bound/2}" y = "${-pos_bound/2}" z = "${rotor_z}" pich = "${opt_pich_2}" yaw = "${opt_yaw_2}"  direction = "-1" />
-  <xacro:propeller_module id = "3" x = "${pos_bound/2}" y = "${pos_bound/2}" z = "${rotor_z}"  pich = "${opt_pich_3}" yaw = "${opt_yaw_3}" direction = "1" />
-  <xacro:propeller_module id = "4" x = "${-pos_bound/2}" y = "${pos_bound/2}" z = "${rotor_z}"  pich = "${opt_pich_4}" yaw = "${opt_yaw_4}"  direction = "-1" />
+  <!-- <xacro:propeller_module id = "1" x = "${-pos_bound/2}" y = "${-pos_bound/2}" z = "${rotor_z}" pich = "${opt_pich_1}" yaw = "${opt_yaw_1}" direction = "1" /> -->
+  <!-- <xacro:propeller_module id = "2" x = "${pos_bound/2}" y = "${-pos_bound/2}" z = "${rotor_z}" pich = "${opt_pich_2}" yaw = "${opt_yaw_2}"  direction = "-1" /> -->
+  <!-- <xacro:propeller_module id = "3" x = "${pos_bound/2}" y = "${pos_bound/2}" z = "${rotor_z}"  pich = "${opt_pich_3}" yaw = "${opt_yaw_3}" direction = "1" /> -->
+  <!-- <xacro:propeller_module id = "4" x = "${-pos_bound/2}" y = "${pos_bound/2}" z = "${rotor_z}"  pich = "${opt_pich_4}" yaw = "${opt_yaw_4}"  direction = "-1" /> -->
+    <xacro:propeller_module id = "1" x = "-0.1044" y = "-0.12014" z = "0.05402" pich = "${-opt_pich_3}" yaw = "${opt_yaw_3}" direction = "1" />
+  <xacro:propeller_module id = "2" x = "0.10705" y = "-0.10827" z = "0.05946" pich = "${-opt_pich_4}" yaw = "${opt_yaw_4}"  direction = "-1" />
+  <xacro:propeller_module id = "3" x = "0.10705" y = "0.10827" z = "0.05402"  pich = "${-opt_pich_1}" yaw = "${opt_yaw_1}" direction = "1" />
+  <xacro:propeller_module id = "4" x = "-0.10705" y = "0.12014" z = "0.05404"  pich = "${-opt_pich_2}" yaw = "${opt_yaw_2}"  direction = "-1" />
 </robot>

File: robots/assemble_quadrotors/urdf/assemble_dual_quadrotors_neutral.urdf.xacro (robot description, xacro)
@@ -154,7 +154,7 @@
   <!-- <xacro:propeller_module id = "3" x = "0.10474" y = "0.10579" z = "0.05404"  pich = "${opt_pich_2}" yaw = "${opt_yaw_2}" direction = "1" /> -->
   <!-- <xacro:propeller_module id = "4" x = "-0.10757" y = "0.12281" z = "0.05404"  pich = "${opt_pich_1}" yaw = "${opt_yaw_1}"  direction = "-1" /> -->
-  <xacro:propeller_module id = "1" x = "-0.104" y = "-0.12" z = "0.05404" pich = "${-opt_pich_3}" yaw = "${opt_yaw_3}" direction = "1" />
-  <xacro:propeller_module id = "2" x = "0.107" y = "-0.11" z = "0.05404" pich = "${-opt_pich_4}" yaw = "${opt_yaw_4}"  direction = "-1" />
-  <xacro:propeller_module id = "3" x = "0.104" y = "0.11" z = "0.05404"  pich = "${-opt_pich_1}" yaw = "${opt_yaw_1}" direction = "1" />
-  <xacro:propeller_module id = "4" x = "-0.107" y = "0.12" z = "0.05404"  pich = "${-opt_pich_2}" yaw = "${opt_yaw_2}"  direction = "-1" />
+  <xacro:propeller_module id = "1" x = "-0.1044" y = "-0.12014" z = "0.05402" pich = "${-opt_pich_3}" yaw = "${opt_yaw_3}" direction = "1" />
+  <xacro:propeller_module id = "2" x = "0.10705" y = "-0.10827" z = "0.05946" pich = "${-opt_pich_4}" yaw = "${opt_yaw_4}"  direction = "-1" />
+  <xacro:propeller_module id = "3" x = "0.10705" y = "0.10827" z = "0.05402"  pich = "${-opt_pich_1}" yaw = "${opt_yaw_1}" direction = "1" />
+  <xacro:propeller_module id = "4" x = "-0.10705" y = "0.12014" z = "0.05404"  pich = "${-opt_pich_2}" yaw = "${opt_yaw_2}"  direction = "-1" />
 </robot>

File: robots/assemble_quadrotors/urdf/assemble_dual_quadrotors_whole.urdf.xacro (robot description, xacro)
@@ -139,5 +139,5 @@
   <!-- spinal -->
   <xacro:extra_module name = "fc" parent = "main_body" visible = "0" >
-    <origin xyz="0 0 0" rpy="0 0 0"/>
+    <origin xyz="-0.2 0 0" rpy="0 0 0"/>
     <inertial>
       <mass value = "0.05" />
@@ -158,11 +158,19 @@
   <!-- <xacro:propeller_module id = "7" x = "-0.30012" y = "-0.12015" z = "0.0521"  pich = "${-opt_pich_3}" yaw = "${opt_yaw_3}" direction = "1" /> -->
   <!-- <xacro:propeller_module id = "8" x = "-0.0886" y = "-0.10827" z = "0.05752"  pich = "${-opt_pich_4}" yaw = "${opt_yaw_4}"  direction = "-1" /> -->
-  <xacro:propeller_module id = "1" x = "0.09" y = "-0.107" z = "0.0521" pich = "${opt_pich_1}" yaw = "${opt_yaw_1}" direction = "1" />
-  <xacro:propeller_module id = "2" x = "0.3" y = "-0.12" z = "0.0521" pich = "${opt_pich_2}" yaw = "${opt_yaw_2}"  direction = "-1" />
-  <xacro:propeller_module id = "3" x = "0.3" y = "0.12" z = "0.0521"  pich = "${opt_pich_3}" yaw = "${opt_yaw_3}" direction = "1" />
-  <xacro:propeller_module id = "4" x = "0.09" y = "0.107" z = "0.0521"  pich = "${opt_pich_4}" yaw = "${opt_yaw_4}"  direction = "-1" />
-  <xacro:propeller_module id = "5" x = "-0.09" y = "0.107" z = "0.0521"  pich = "${-opt_pich_1}" yaw = "${opt_yaw_1}" direction = "1" />
-  <xacro:propeller_module id = "6" x = "-0.3" y = "0.12" z = "0.0521"  pich = "${-opt_pich_2}" yaw = "${opt_yaw_2}" direction = "-1" />
-  <xacro:propeller_module id = "7" x = "-0.3" y = "-0.12" z = "0.0521"  pich = "${-opt_pich_3}" yaw = "${opt_yaw_3}" direction = "1" />
-  <xacro:propeller_module id = "8" x = "-0.09" y = "-0.107" z = "0.0521"  pich = "${-opt_pich_4}" yaw = "${opt_yaw_4}"  direction = "-1" />
+  <!-- <xacro:propeller_module id = "1" x = "0.08961" y = "-0.10707" z = "0.0546" pich = "${opt_pich_1}" yaw = "${opt_yaw_1}" direction = "1" /> -->
+  <!-- <xacro:propeller_module id = "2" x = "0.30328" y = "-0.12278" z = "0.05074" pich = "${opt_pich_2}" yaw = "${opt_yaw_2}"  direction = "-1" /> -->
+  <!-- <xacro:propeller_module id = "3" x = "0.30328" y = "0.12278" z = "0.05074"  pich = "${opt_pich_3}" yaw = "${opt_yaw_3}" direction = "1" /> -->
+  <!-- <xacro:propeller_module id = "4" x = "0.08961" y = "0.10707" z = "0.05074"  pich = "${opt_pich_4}" yaw = "${opt_yaw_4}"  direction = "-1" /> -->
+  <!-- <xacro:propeller_module id = "5" x = "-0.08961" y = "0.10707" z = "0.0521"  pich = "${-opt_pich_1}" yaw = "${opt_yaw_1}" direction = "1" /> -->
+  <!-- <xacro:propeller_module id = "6" x = "-0.30328" y = "0.12278" z = "0.0521"  pich = "${-opt_pich_2}" yaw = "${opt_yaw_2}" direction = "-1" /> -->
+  <!-- <xacro:propeller_module id = "7" x = "-0.30328" y = "-0.12278" z = "0.0521"  pich = "${-opt_pich_3}" yaw = "${opt_yaw_3}" direction = "1" /> -->
+  <!-- <xacro:propeller_module id = "8" x = "-0.08961" y = "-0.10707" z = "0.0521"  pich = "${-opt_pich_4}" yaw = "${opt_yaw_4}"  direction = "-1" /> -->
+  <xacro:propeller_module id = "1" x = "-0.30328" y = "-0.12278" z = "0.0521"  pich = "${-opt_pich_3}" yaw = "${opt_yaw_3}" direction = "1" />
+  <xacro:propeller_module id = "2" x = "-0.08961" y = "-0.10707" z = "0.0521"  pich = "${-opt_pich_4}" yaw = "${opt_yaw_4}"  direction = "-1" />
+  <xacro:propeller_module id = "3" x = "-0.08961" y = "0.10707" z = "0.0521"  pich = "${-opt_pich_1}" yaw = "${opt_yaw_1}" direction = "1" />
+  <xacro:propeller_module id = "4" x = "-0.30328" y = "0.12278" z = "0.0521"  pich = "${-opt_pich_2}" yaw = "${opt_yaw_2}" direction = "-1" />
+  <xacro:propeller_module id = "5" x = "0.30328" y = "0.12278" z = "0.05074"  pich = "${opt_pich_3}" yaw = "${opt_yaw_3}" direction = "1" />
+  <xacro:propeller_module id = "6" x = "0.08961" y = "0.10707" z = "0.05074"  pich = "${opt_pich_4}" yaw = "${opt_yaw_4}"  direction = "-1" />
+  <xacro:propeller_module id = "7" x = "0.08961" y = "-0.10707" z = "0.0546" pich = "${opt_pich_1}" yaw = "${opt_yaw_1}" direction = "1" />
+  <xacro:propeller_module id = "8" x = "0.30328" y = "-0.12278" z = "0.05074" pich = "${opt_pich_2}" yaw = "${opt_yaw_2}"  direction = "-1" />
 </robot>

Commit message: [URDF] modification for the inertia of female unit

File: robots/assemble_quadrotors/urdf/assemble_dual_quadrotors_female.urdf.xacro (robot description, xacro)
@@ -109,10 +109,10 @@
   <link name="main_body">
     <inertial>
-      <mass value = "0.75397839" />
-      <origin xyz="0 0 0 " rpy="0 0 0"/>
+      <mass value = "0.9251" />
+      <origin xyz="0.007 0.0 0.04 " rpy="0 0 0"/>
       <inertia
-          ixx="0.00523481" ixy="-0.00011631" ixz="-0.00040281"
-          iyy="0.00740303" iyz="-0.00003402"
-          izz="0.01114830"/>
+          ixx="0.00621238" ixy="-0.00001138" ixz="-0.00041267"
+          iyy="0.00844836" iyz="-0.00001426"
+          izz="0.01253637"/>
     </inertial>
     <visual>

Commit message: [URDF] rechanged male inertia

File: robots/assemble_quadrotors/urdf/assemble_dual_quadrotors_female.urdf.xacro (robot description, xacro)
@@ -110,5 +110,5 @@
     <inertial>
       <mass value = "0.9251" />
-      <origin xyz="0.007 0.0 0.04 " rpy="0 0 0"/>
+      <origin xyz="0.007 0.0 0.02 " rpy="0 0 0"/>
       <inertia
           ixx="0.00621238" ixy="-0.00001138" ixz="-0.00041267"
