Commit message: [Model and Navigaiton] workaround activation of assemble model

File: robots/assemble_quadrotors/urdf/assemble_dual_quadrotors_female.urdf.xacro (robot description, xacro)
@@ -109,5 +109,5 @@
   <link name="main_body">
     <inertial>
-      <mass value = "0.9251" />
+      <mass value = "0.8751" />
       <origin xyz="0.007 0.0 0.02 " rpy="0 0 0"/>
       <inertia
@@ -142,7 +142,7 @@
   </xacro:extra_module>
   <!-- propellers -->
-  <xacro:propeller_module id = "1" x = "-0.1044" y = "-0.12014" z = "0.05402" pich = "${-opt_pich_3}" yaw = "${opt_yaw_3}" direction = "1" />
-  <xacro:propeller_module id = "2" x = "0.10705" y = "-0.10827" z = "0.05946" pich = "${-opt_pich_4}" yaw = "${opt_yaw_4}"  direction = "-1" />
-  <xacro:propeller_module id = "3" x = "0.10705" y = "0.10827" z = "0.05402"  pich = "${-opt_pich_1}" yaw = "${opt_yaw_1}" direction = "1" />
-  <xacro:propeller_module id = "4" x = "-0.10705" y = "0.12014" z = "0.05404"  pich = "${-opt_pich_2}" yaw = "${opt_yaw_2}"  direction = "-1" />
+  <xacro:propeller_module id = "1" x = "-0.10754" y = "-0.12284" z = "0.05287" pich = "${-opt_pich_3}" yaw = "${opt_yaw_3}" direction = "1" />
+  <xacro:propeller_module id = "2" x = "0.10610" y = "-0.10682" z = "0.05662" pich = "${-opt_pich_4}" yaw = "${opt_yaw_4}"  direction = "-1" />
+  <xacro:propeller_module id = "3" x = "0.10618" y = "0.10708" z = "0.05674"  pich = "${-opt_pich_1}" yaw = "${opt_yaw_1}" direction = "1" />
+  <xacro:propeller_module id = "4" x = "-0.10744" y = "0.12274" z = "0.05289"  pich = "${-opt_pich_2}" yaw = "${opt_yaw_2}"  direction = "-1" />
 </robot>

File: robots/assemble_quadrotors/urdf/assemble_dual_quadrotors_male.urdf.xacro (robot description, xacro)
@@ -6,15 +6,4 @@
   <thrust_link name="thrust" />
   <!-- kinematics [m] -->
-  <!-- <xacro:property name="pos_bound" value="${0.22628}" /> -->
-  <!-- <xacro:property name="center_dis" value="${0.393}" /> -->
-  <!-- <xacro:property name="rotor_z" value="${0.05}" /> -->
-  <!-- <xacro:property name="opt_pich_1" value="${0.523525}" /> -->
-  <!-- <xacro:property name="opt_yaw_1" value="${0.73108}" /> -->
-  <!-- <xacro:property name="opt_pich_2" value="${0.523535}" /> -->
-  <!-- <xacro:property name="opt_yaw_2" value="${-2.08113}" /> -->
-  <!-- <xacro:property name="opt_pich_3" value="${0.523595}" /> -->
-  <!-- <xacro:property name="opt_yaw_3" value="${2.4662}" /> -->
-  <!-- <xacro:property name="opt_pich_4" value="${0.348489}" /> -->
-  <!-- <xacro:property name="opt_yaw_4" value="${-0.673131}" /> -->
   <xacro:property name="pos_bound" value="${0.22628}" />
   <xacro:property name="center_dis" value="${0.393}" />
@@ -120,5 +109,5 @@
   <link name="main_body">
     <inertial>
-      <mass value = "0.99287590" />
+      <mass value = "0.94287590" />
       <origin xyz="0.0209037 -0.00157892 0.00576541" rpy="0 0 0"/>
     <inertia
@@ -153,11 +142,7 @@
   </xacro:extra_module>
   <!-- propellers -->
-  <!-- <xacro:propeller_module id = "1" x = "${-pos_bound/2}" y = "${-pos_bound/2}" z = "${rotor_z}" pich = "${opt_pich_1}" yaw = "${opt_yaw_1}" direction = "1" /> -->
-  <!-- <xacro:propeller_module id = "2" x = "${pos_bound/2}" y = "${-pos_bound/2}" z = "${rotor_z}" pich = "${opt_pich_2}" yaw = "${opt_yaw_2}"  direction = "-1" /> -->
-  <!-- <xacro:propeller_module id = "3" x = "${pos_bound/2}" y = "${pos_bound/2}" z = "${rotor_z}"  pich = "${opt_pich_3}" yaw = "${opt_yaw_3}" direction = "1" /> -->
-  <!-- <xacro:propeller_module id = "4" x = "${-pos_bound/2}" y = "${pos_bound/2}" z = "${rotor_z}"  pich = "${opt_pich_4}" yaw = "${opt_yaw_4}"  direction = "-1" /> -->
-    <xacro:propeller_module id = "1" x = "-0.1044" y = "-0.12014" z = "0.05402" pich = "${-opt_pich_3}" yaw = "${opt_yaw_3}" direction = "1" />
-  <xacro:propeller_module id = "2" x = "0.10705" y = "-0.10827" z = "0.05946" pich = "${-opt_pich_4}" yaw = "${opt_yaw_4}"  direction = "-1" />
-  <xacro:propeller_module id = "3" x = "0.10705" y = "0.10827" z = "0.05402"  pich = "${-opt_pich_1}" yaw = "${opt_yaw_1}" direction = "1" />
-  <xacro:propeller_module id = "4" x = "-0.10705" y = "0.12014" z = "0.05404"  pich = "${-opt_pich_2}" yaw = "${opt_yaw_2}"  direction = "-1" />
+  <xacro:propeller_module id = "1" x = "-0.10754" y = "-0.12284" z = "0.05287" pich = "${-opt_pich_3}" yaw = "${opt_yaw_3}" direction = "1" />
+  <xacro:propeller_module id = "2" x = "0.10610" y = "-0.10682" z = "0.05662" pich = "${-opt_pich_4}" yaw = "${opt_yaw_4}"  direction = "-1" />
+  <xacro:propeller_module id = "3" x = "0.10618" y = "0.10708" z = "0.05674"  pich = "${-opt_pich_1}" yaw = "${opt_yaw_1}" direction = "1" />
+  <xacro:propeller_module id = "4" x = "-0.10744" y = "0.12274" z = "0.05289"  pich = "${-opt_pich_2}" yaw = "${opt_yaw_2}"  direction = "-1" />
 </robot>

File: robots/assemble_quadrotors/urdf/assemble_dual_quadrotors_whole.urdf.xacro (robot description, xacro)
@@ -7,14 +7,6 @@
   <!-- kinematics [m] -->
   <xacro:property name="pos_bound" value="${0.22628}" />
-  <xacro:property name="center_dis" value="${0.393}" />
-  <xacro:property name="rotor_z" value="${0.050}" />
-  <xacro:property name="opt_pich_1" value="${0.523525}" />
-  <xacro:property name="opt_yaw_1" value="${0.73108}" />
-  <!-- <xacro:property name="opt_pich_2" value="${0.523535}" /> -->
-  <!-- <xacro:property name="opt_yaw_2" value="${-2.08113}" /> -->
-  <!-- <xacro:property name="opt_pich_3" value="${0.523595}" /> -->
-  <!-- <xacro:property name="opt_yaw_3" value="${2.4662}" /> -->
-  <!-- <xacro:property name="opt_pich_4" value="${0.348489}" /> -->
-  <!-- <xacro:property name="opt_yaw_4" value="${-0.673131}" /> -->
+  <xacro:property name="center_dis_x" value="${0.199}" />
+  <xacro:property name="rotor_z" value="${0.052}" />
   <xacro:property name="opt_pich_1" value="${0.45}" />
   <xacro:property name="opt_yaw_1" value="${0.73108}" />
@@ -117,15 +109,15 @@
   <link name="main_body">
     <inertial>
-      <mass value = "1.54552806" />
-      <origin xyz="0 0 0" rpy="0 0 0"/>
+      <mass value = "1.84719908" />
+      <origin xyz="-0.00401288 0.00002524 0.00751852" rpy="0 0 0"/>
       <inertia
-          ixx="0.01124041" ixy="-0.00026951" ixz="-0.00026951"
-          iyy="0.06648421" iyz="0.00007432"
-          izz="0.07433712"/>
+          ixx="0.01198006" ixy="0.00062162" ixz="0.00027258"
+          iyy="0.08096541" iyz="-0.00000195"
+          izz="0.08846491"/>
     </inertial>
     <visual>
       <origin rpy="0 0 0" xyz="0 0 0"/>
       <geometry>
-        <mesh filename="package://assemble_quadrotors/urdf/mesh/Assemble_dual_quadrotors_v3_whole.STL"/>
+        <mesh filename="package://assemble_quadrotors/urdf/mesh/Assemble_dual_quadrotors_v4.STL"/>
       </geometry>
     </visual>
@@ -139,5 +131,5 @@
   <!-- spinal -->
   <xacro:extra_module name = "fc" parent = "main_body" visible = "0" >
-    <origin xyz="-0.2 0 0" rpy="0 0 0"/>
+    <origin xyz="-0.2 0.0 0.0" rpy="0 0 0"/>
     <inertial>
       <mass value = "0.05" />
@@ -150,27 +142,19 @@
   </xacro:extra_module>
   <!-- propellers -->
-  <!-- <xacro:propeller_module id = "1" x = "0.09099" y = "-0.10578" z = "0.0521" pich = "${opt_pich_1}" yaw = "${opt_yaw_1}" direction = "1" /> -->
-  <!-- <xacro:propeller_module id = "2" x = "0.30329" y = "-0.1228" z = "0.0521" pich = "${opt_pich_2}" yaw = "${opt_yaw_2}"  direction = "-1" /> -->
-  <!-- <xacro:propeller_module id = "3" x = "0.30012" y = "0.12015" z = "0.0521"  pich = "${opt_pich_3}" yaw = "${opt_yaw_3}" direction = "1" /> -->
-  <!-- <xacro:propeller_module id = "4" x = "0.0886" y = "0.10827" z = "0.05752"  pich = "${opt_pich_4}" yaw = "${opt_yaw_4}"  direction = "-1" /> -->
-  <!-- <xacro:propeller_module id = "5" x = "-0.09099" y = "0.10578" z = "0.0521"  pich = "${-opt_pich_1}" yaw = "${opt_yaw_1}" direction = "1" /> -->
-  <!-- <xacro:propeller_module id = "6" x = "-0.30329" y = "0.1228" z = "0.0521"  pich = "${-opt_pich_2}" yaw = "${opt_yaw_2}" direction = "-1" /> -->
-  <!-- <xacro:propeller_module id = "7" x = "-0.30012" y = "-0.12015" z = "0.0521"  pich = "${-opt_pich_3}" yaw = "${opt_yaw_3}" direction = "1" /> -->
-  <!-- <xacro:propeller_module id = "8" x = "-0.0886" y = "-0.10827" z = "0.05752"  pich = "${-opt_pich_4}" yaw = "${opt_yaw_4}"  direction = "-1" /> -->
-  <!-- <xacro:propeller_module id = "1" x = "0.08961" y = "-0.10707" z = "0.0546" pich = "${opt_pich_1}" yaw = "${opt_yaw_1}" direction = "1" /> -->
-  <!-- <xacro:propeller_module id = "2" x = "0.30328" y = "-0.12278" z = "0.05074" pich = "${opt_pich_2}" yaw = "${opt_yaw_2}"  direction = "-1" /> -->
-  <!-- <xacro:propeller_module id = "3" x = "0.30328" y = "0.12278" z = "0.05074"  pich = "${opt_pich_3}" yaw = "${opt_yaw_3}" direction = "1" /> -->
-  <!-- <xacro:propeller_module id = "4" x = "0.08961" y = "0.10707" z = "0.05074"  pich = "${opt_pich_4}" yaw = "${opt_yaw_4}"  direction = "-1" /> -->
-  <!-- <xacro:propeller_module id = "5" x = "-0.08961" y = "0.10707" z = "0.0521"  pich = "${-opt_pich_1}" yaw = "${opt_yaw_1}" direction = "1" /> -->
-  <!-- <xacro:propeller_module id = "6" x = "-0.30328" y = "0.12278" z = "0.0521"  pich = "${-opt_pich_2}" yaw = "${opt_yaw_2}" direction = "-1" /> -->
-  <!-- <xacro:propeller_module id = "7" x = "-0.30328" y = "-0.12278" z = "0.0521"  pich = "${-opt_pich_3}" yaw = "${opt_yaw_3}" direction = "1" /> -->
-  <!-- <xacro:propeller_module id = "8" x = "-0.08961" y = "-0.10707" z = "0.0521"  pich = "${-opt_pich_4}" yaw = "${opt_yaw_4}"  direction = "-1" /> -->
-  <xacro:propeller_module id = "1" x = "-0.30328" y = "-0.12278" z = "0.0521"  pich = "${-opt_pich_3}" yaw = "${opt_yaw_3}" direction = "1" />
-  <xacro:propeller_module id = "2" x = "-0.08961" y = "-0.10707" z = "0.0521"  pich = "${-opt_pich_4}" yaw = "${opt_yaw_4}"  direction = "-1" />
-  <xacro:propeller_module id = "3" x = "-0.08961" y = "0.10707" z = "0.0521"  pich = "${-opt_pich_1}" yaw = "${opt_yaw_1}" direction = "1" />
-  <xacro:propeller_module id = "4" x = "-0.30328" y = "0.12278" z = "0.0521"  pich = "${-opt_pich_2}" yaw = "${opt_yaw_2}" direction = "-1" />
-  <xacro:propeller_module id = "5" x = "0.30328" y = "0.12278" z = "0.05074"  pich = "${opt_pich_3}" yaw = "${opt_yaw_3}" direction = "1" />
-  <xacro:propeller_module id = "6" x = "0.08961" y = "0.10707" z = "0.05074"  pich = "${opt_pich_4}" yaw = "${opt_yaw_4}"  direction = "-1" />
-  <xacro:propeller_module id = "7" x = "0.08961" y = "-0.10707" z = "0.0546" pich = "${opt_pich_1}" yaw = "${opt_yaw_1}" direction = "1" />
-  <xacro:propeller_module id = "8" x = "0.30328" y = "-0.12278" z = "0.05074" pich = "${opt_pich_2}" yaw = "${opt_yaw_2}"  direction = "-1" />
+  <!-- <xacro:propeller_module id = "1" x = "-0.30328" y = "-0.12278" z = "0.0521"  pich = "${-opt_pich_3}" yaw = "${opt_yaw_3}" direction = "1" /> -->
+  <!-- <xacro:propeller_module id = "2" x = "-0.08961" y = "-0.10707" z = "0.0521"  pich = "${-opt_pich_4}" yaw = "${opt_yaw_4}"  direction = "-1" /> -->
+  <!-- <xacro:propeller_module id = "3" x = "-0.08961" y = "0.10707" z = "0.0521"  pich = "${-opt_pich_1}" yaw = "${opt_yaw_1}" direction = "1" /> -->
+  <!-- <xacro:propeller_module id = "4" x = "-0.30328" y = "0.12278" z = "0.0521"  pich = "${-opt_pich_2}" yaw = "${opt_yaw_2}" direction = "-1" /> -->
+  <!-- <xacro:propeller_module id = "5" x = "0.30328" y = "0.12278" z = "0.05074"  pich = "${opt_pich_3}" yaw = "${opt_yaw_3}" direction = "1" /> -->
+  <!-- <xacro:propeller_module id = "6" x = "0.08961" y = "0.10707" z = "0.05074"  pich = "${opt_pich_4}" yaw = "${opt_yaw_4}"  direction = "-1" /> -->
+  <!-- <xacro:propeller_module id = "7" x = "0.08961" y = "-0.10707" z = "0.0546" pich = "${opt_pich_1}" yaw = "${opt_yaw_1}" direction = "1" /> -->
+  <!-- <xacro:propeller_module id = "8" x = "0.30328" y = "-0.12278" z = "0.05074" pich = "${opt_pich_2}" yaw = "${opt_yaw_2}"  direction = "-1" /> -->
+  <xacro:propeller_module id = "1" x = "${-0.10754 - center_dis_x}" y = "-0.12284" z = "0.05287" pich = "${-opt_pich_3}" yaw = "${opt_yaw_3}" direction = "1" />
+  <xacro:propeller_module id = "2" x = "${0.10610 - center_dis_x}" y = "-0.10682" z = "0.05662" pich = "${-opt_pich_4}" yaw = "${opt_yaw_4}"  direction = "-1" />
+  <xacro:propeller_module id = "3" x = "${0.10618 - center_dis_x}" y = "0.10708" z = "0.05674"  pich = "${-opt_pich_1}" yaw = "${opt_yaw_1}" direction = "1" />
+  <xacro:propeller_module id = "4" x = "${-0.10744 - center_dis_x}" y = "0.12274" z = "0.05289"  pich = "${-opt_pich_2}" yaw = "${opt_yaw_2}"  direction = "-1" />
+  <xacro:propeller_module id = "5" x = "${0.10754 + center_dis_x}" y = "0.12284" z = "0.05287" pich = "${opt_pich_3}" yaw = "${opt_yaw_3}" direction = "1" />
+  <xacro:propeller_module id = "6" x = "${-0.10610 + center_dis_x}" y = "0.10682" z = "0.05662" pich = "${opt_pich_4}" yaw = "${opt_yaw_4}"  direction = "-1" />
+  <xacro:propeller_module id = "7" x = "${-0.10618 + center_dis_x}" y = "-0.10708" z = "0.05674"  pich = "${opt_pich_1}" yaw = "${opt_yaw_1}" direction = "1" />
+  <xacro:propeller_module id = "8" x = "${0.10744 + center_dis_x}" y = "-0.12274" z = "0.05289"  pich = "${opt_pich_2}" yaw = "${opt_yaw_2}"  direction = "-1" />
 </robot>

Commit message: [URDF] corrected mass values of male and female

File: robots/assemble_quadrotors/urdf/assemble_dual_quadrotors_female.urdf.xacro (robot description, xacro)
@@ -109,5 +109,5 @@
   <link name="main_body">
     <inertial>
-      <mass value = "0.8751" />
+      <mass value = "0.9685" />
       <origin xyz="0.007 0.0 0.02 " rpy="0 0 0"/>
       <inertia

File: robots/assemble_quadrotors/urdf/assemble_dual_quadrotors_male.urdf.xacro (robot description, xacro)
@@ -109,5 +109,5 @@
   <link name="main_body">
     <inertial>
-      <mass value = "0.94287590" />
+      <mass value = "1.1455" />
       <origin xyz="0.0209037 -0.00157892 0.00576541" rpy="0 0 0"/>
     <inertia

File: robots/assemble_quadrotors/urdf/assemble_dual_quadrotors_whole_female.urdf.xacro (robot description, xacro)
@@ -109,5 +109,5 @@
   <link name="main_body">
     <inertial>
-      <mass value = "1.84719908" />
+      <mass value = "2.114" />
       <origin xyz="0.00401288 0.00002524 0.00751852" rpy="0 0 0"/>
       <inertia

File: robots/assemble_quadrotors/urdf/assemble_dual_quadrotors_whole_male.urdf.xacro (robot description, xacro)
@@ -109,5 +109,5 @@
   <link name="main_body">
     <inertial>
-      <mass value = "1.84719908" />
+      <mass value = "2.114" />
       <origin xyz="-0.00401288 0.00002524 0.00751852" rpy="0 0 0"/>
       <inertia

Commit message: [URDF] modified male and female models

File: robots/assemble_quadrotors/urdf/assemble_dual_quadrotors_female.urdf.xacro (robot description, xacro)
@@ -109,10 +109,10 @@
   <link name="main_body">
     <inertial>
-      <mass value = "0.9685" />
-      <origin xyz="0.007 0.0 0.02 " rpy="0 0 0"/>
+      <mass value = "1.0725" />
+      <origin xyz="-0.0163497 -0.00181591 0.0065744 " rpy="0 0 0"/>
       <inertia
-          ixx="0.00621238" ixy="-0.00001138" ixz="-0.00041267"
-          iyy="0.00844836" iyz="-0.00001426"
-          izz="0.01253637"/>
+          ixx="0.00605748" ixy="-0.00005473" ixz="0.00028180"
+          iyy="0.01078895" iyz="-0.00001861"
+          izz="0.01463121"/>
     </inertial>
     <visual>

File: robots/assemble_quadrotors/urdf/assemble_dual_quadrotors_male.urdf.xacro (robot description, xacro)
@@ -109,10 +109,10 @@
   <link name="main_body">
     <inertial>
-      <mass value = "1.1455" />
-      <origin xyz="0.0209037 -0.00157892 0.00576541" rpy="0 0 0"/>
+      <mass value = "1.2495" />
+      <origin xyz="-0.00957258 -0.00152585 0.00321411" rpy="0 0 0"/>
     <inertia
-        ixx="0.00608728" ixy="0.00003070" ixz="-0.00079536"
-        iyy="0.00932989" iyz="-0.00002784"
-        izz="0.01298518"/>
+        ixx="0.00624824" ixy="-0.00002383" ixz="-0.00008370"
+        iyy="0.01304324" iyz="-0.00002877"
+        izz="0.01671753"/>
     </inertial>
     <visual>

Commit message: [URDF] additional weight on female

File: robots/assemble_quadrotors/urdf/assemble_dual_quadrotors_female.urdf.xacro (robot description, xacro)
@@ -109,10 +109,10 @@
   <link name="main_body">
     <inertial>
-      <mass value = "1.0725" />
-      <origin xyz="-0.0163497 -0.00181591 0.0065744 " rpy="0 0 0"/>
+      <mass value = "1.2545" />
+      <origin xyz="-0.02178050 0.0 0.00309236 " rpy="0 0 0"/>
       <inertia
-          ixx="0.00605748" ixy="-0.00005473" ixz="0.00028180"
-          iyy="0.01078895" iyz="-0.00001861"
-          izz="0.01463121"/>
+          ixx="0.00631767" ixy="-0.00006783" ixz="0.00039834"
+          iyy="0.01106646" iyz="-0.00002838"
+          izz="0.01499360"/>
     </inertial>
     <visual>

File: robots/assemble_quadrotors/urdf/assemble_dual_quadrotors_male.urdf.xacro (robot description, xacro)
@@ -110,5 +110,5 @@
     <inertial>
       <mass value = "1.2495" />
-      <origin xyz="-0.00957258 -0.00152585 0.00321411" rpy="0 0 0"/>
+      <origin xyz="-0.00957258 0.0 0.00321411" rpy="0 0 0"/>
     <inertia
         ixx="0.00624824" ixy="-0.00002383" ixz="-0.00008370"

File: robots/assemble_quadrotors/urdf/assemble_dual_quadrotors_whole_female.urdf.xacro (robot description, xacro)
@@ -109,12 +109,12 @@
   <link name="main_body">
     <inertial>
-      <mass value = "2.318" />
+      <mass value = "2.5" />
       <!-- <origin xyz="0.00401288 0.00002524 0.00751852" rpy="0 0 0"/> -->
-      <origin xyz="0.00363315 -0.00001636 0.00477654" rpy="0 0 0"/> <!-- for wierd -->
+      <origin xyz="-0.01665965 0.00002872 0.00310773" rpy="0 0 0"/> <!-- for wierd -->
       <!-- <origin xyz="0.0 0.0 0.0" rpy="0 0 0"/> -->
       <inertia
-          ixx="0.01231937" ixy="0.00082883" ixz="-0.00028830"
-          iyy="0.11563003" iyz="0.00000115"
-          izz="0.12314029"/>
+          ixx="0.01257219" ixy="0.00079619" ixz="0.00057445"
+          iyy="0.12647091" iyz="-0.00000082"
+          izz="0.13407114"/>
     </inertial>
     <visual>

File: robots/assemble_quadrotors/urdf/assemble_dual_quadrotors_whole_male.urdf.xacro (robot description, xacro)
@@ -109,12 +109,12 @@
   <link name="main_body">
     <inertial>
-      <mass value = "2.318" />
+      <mass value = "2.5" />
       <!-- <origin xyz="-0.00401288 0.00002524 0.00751852" rpy="0 0 0"/> -->
-      <origin xyz="-0.00363315 0.00001636 0.00477654" rpy="0 0 0"/> <!-- for wierd -->
+      <origin xyz="0.01665965 -0.00002872 0.00310773" rpy="0 0 0"/> <!-- for wierd -->
       <!-- <origin xyz="0.0 0.00 0.00" rpy="0 0 0"/> -->
       <inertia
-          ixx="0.01231937" ixy="0.00082883" ixz="0.00028830"
-          iyy="0.11563003" iyz="-0.00000115"
-          izz="0.12314029"/>
+          ixx="0.01257219" ixy="0.00079619" ixz="-0.00057445"
+          iyy="0.12647091" iyz="0.00000082"
+          izz="0.13407114"/>
     </inertial>
     <visual>
