Commit message: [URDF]modified whole urdf for battery mode

File: robots/assemble_quadrotors/urdf/assemble_dual_quadrotors_whole_female_mag.urdf.xacro (robot description, xacro)
@@ -109,10 +109,10 @@
   <link name="main_body">
     <inertial>
-      <mass value = "2.46" />
-      <origin xyz="-0.00186 0.00003441 -0.00128" rpy="0 0 0"/>
+      <mass value = "2.462" />
+      <origin xyz="-0.001 0.000 -0.001" rpy="0 0 0"/>
       <inertia
-          ixx="0.0125" ixy="0.000837" ixz="0.000138"
-          iyy="0.125" iyz="-0.00000554"
-          izz="0.132"/>
+          ixx="0.013" ixy="-0.001" ixz="0.00"
+          iyy="0.119" iyz="0.000"
+          izz="0.126"/>
     </inertial>
     <visual>

File: robots/assemble_quadrotors/urdf/assemble_dual_quadrotors_whole_male_mag.urdf.xacro (robot description, xacro)
@@ -109,10 +109,10 @@
   <link name="main_body">
     <inertial>
-      <mass value = "2.492" />
-      <origin xyz="0.002 0.000 0.000" rpy="0 0 0"/>
+      <mass value = "2.462" />
+      <origin xyz="0.001 0.000 -0.001" rpy="0 0 0"/>
       <inertia
-          ixx="0.013" ixy="0.001" ixz="0.00"
-          iyy="0.133" iyz="0.000"
-          izz="0.14"/>
+          ixx="0.013" ixy="-0.001" ixz="0.00"
+          iyy="0.119" iyz="0.000"
+          izz="0.126"/>
     </inertial>
     <visual>
