Commit message: [URDF]modified female urdf nad related ones

File: robots/assemble_quadrotors/urdf/assemble_dual_quadrotors_female_mag.urdf.xacro (robot description, xacro)
@@ -109,10 +109,16 @@
   <link name="main_body">
     <inertial>
-      <mass value = "1.427857" />
-      <origin xyz="-0.00884209 -0.00096336 -0.00122007 " rpy="0 0 0"/>
+      <!-- <mass value = "1.427857" /> -->
+      <!-- <origin xyz="-0.00884209 -0.00096336 -0.00122007 " rpy="0 0 0"/> -->
+      <!-- <inertia -->
+      <!--     ixx="0.00716924" ixy="0.00006933" ixz="-0.00025713" -->
+      <!--     iyy="0.01398491" iyz="-0.00005390" -->
+      <!--     izz="0.01819428"/> -->
+      <mass value = "1.247857" />
+      <origin xyz="-0.00279206 -0.00110497 0.00095251 " rpy="0 0 0"/>
       <inertia
-          ixx="0.00716924" ixy="0.00006933" ixz="-0.00025713"
-          iyy="0.01398491" iyz="-0.00005390"
-          izz="0.01819428"/>
+          ixx="0.00689482" ixy="0.00007765" ixz="-0.00038481"
+          iyy="0.01355710" iyz="-0.00005091"
+          izz="0.01760133"/>
     </inertial>
     <visual>

File: robots/assemble_quadrotors/urdf/assemble_dual_quadrotors_whole_female_mag.urdf.xacro (robot description, xacro)
@@ -109,10 +109,10 @@
   <link name="main_body">
     <inertial>
-      <mass value = "2.69133021" />
-      <origin xyz="-0.01819575 0.00020102 -0.00057410" rpy="0 0 0"/>
+      <mass value = "2.50834021" />
+      <origin xyz="-0.00140155 0.00021569 0.00055126" rpy="0 0 0"/>
       <inertia
-          ixx="0.01411616" ixy="0.00077103" ixz="0.00081566"
-          iyy="0.13743779" iyz="-0.00001865"
-          izz="0.14660374"/>
+          ixx="0.01384106" ixy="0.00076195" ixz="0.00011842"
+          iyy="0.12795959" iyz="-0.00001926"
+          izz="0.13596145"/>
     </inertial>
     <visual>

File: robots/assemble_quadrotors/urdf/assemble_dual_quadrotors_whole_male_mag.urdf.xacro (robot description, xacro)
@@ -109,10 +109,10 @@
   <link name="main_body">
     <inertial>
-      <mass value = "2.69133021" />
-      <origin xyz="0.01819575 -0.00020102 -0.00057410" rpy="0 0 0"/>
+      <mass value = "2.50834021" />
+      <origin xyz="0.00140155 -0.00021569 0.00055126" rpy="0 0 0"/>
       <inertia
-          ixx="0.01411616" ixy="0.00077103" ixz="-0.00081566"
-          iyy="0.13743779" iyz="0.00001865"
-          izz="0.14660374"/>
+          ixx="0.01384106" ixy="0.00076195" ixz="-0.00011842"
+          iyy="0.12795959" iyz="0.00001926"
+          izz="0.13596145"/>
     </inertial>
     <visual>

Commit message: [URDF][Motor]workaround 6inch propeller

File: robots/assemble_quadrotors/urdf/assemble_dual_quadrotors_female_mag.urdf.xacro (robot description, xacro)
@@ -109,16 +109,10 @@
   <link name="main_body">
     <inertial>
-      <!-- <mass value = "1.427857" /> -->
-      <!-- <origin xyz="-0.00884209 -0.00096336 -0.00122007 " rpy="0 0 0"/> -->
-      <!-- <inertia -->
-      <!--     ixx="0.00716924" ixy="0.00006933" ixz="-0.00025713" -->
-      <!--     iyy="0.01398491" iyz="-0.00005390" -->
-      <!--     izz="0.01819428"/> -->
-      <mass value = "1.247857" />
-      <origin xyz="-0.00279206 -0.00110497 0.00095251 " rpy="0 0 0"/>
+      <mass value = "1.2080" />
+      <origin xyz="-0.002865 -0.001183 -0.00076 " rpy="0 0 0"/>
       <inertia
-          ixx="0.00689482" ixy="0.00007765" ixz="-0.00038481"
-          iyy="0.01355710" iyz="-0.00005091"
-          izz="0.01760133"/>
+          ixx="0.006072" ixy="0.00007563" ixz="-0.000430"
+          iyy="0.012790" iyz="-0.00005"
+          izz="0.01629"/>
     </inertial>
     <visual>

File: robots/assemble_quadrotors/urdf/assemble_dual_quadrotors_male_mag.urdf.xacro (robot description, xacro)
@@ -109,10 +109,10 @@
   <link name="main_body">
     <inertial>
-      <mass value = "1.26347288" />
-      <origin xyz="0.00295047 -0.00151693 0.00015592" rpy="0 0 0"/>
+      <mass value = "1.2266" />
+      <origin xyz="0.0030 -0.0016 -0.00015" rpy="0 0 0"/>
     <inertia
-        ixx="0.00694153" ixy="0.00003221" ixz="-0.00070136"
-        iyy="0.01575032" iyz="-0.00003297"
-        izz="0.01974271"/>
+        ixx="0.00611" ixy="0.0000" ixz="-0.00073"
+        iyy="0.01498" iyz="-0.0000"
+        izz="0.01839"/>
     </inertial>
     <visual>

File: robots/assemble_quadrotors/urdf/assemble_dual_quadrotors_whole_female_mag.urdf.xacro (robot description, xacro)
@@ -109,10 +109,10 @@
   <link name="main_body">
     <inertial>
-      <mass value = "2.50834021" />
-      <origin xyz="-0.00140155 0.00021569 0.00055126" rpy="0 0 0"/>
+      <mass value = "2.4347" />
+      <origin xyz="-0.00144388 0.000222 -0.001163" rpy="0 0 0"/>
       <inertia
-          ixx="0.01384106" ixy="0.00076195" ixz="0.00011842"
-          iyy="0.12795959" iyz="-0.00001926"
-          izz="0.13596145"/>
+          ixx="0.01219350" ixy="0.00078" ixz="0.000112"
+          iyy="0.12351" iyz="-0.00001833"
+          izz="0.13043"/>
     </inertial>
     <visual>

File: robots/assemble_quadrotors/urdf/assemble_dual_quadrotors_whole_male_mag.urdf.xacro (robot description, xacro)
@@ -109,10 +109,10 @@
   <link name="main_body">
     <inertial>
-      <mass value = "2.50834021" />
-      <origin xyz="0.00140155 -0.00021569 0.00055126" rpy="0 0 0"/>
+      <mass value = "2.4347" />
+      <origin xyz="0.00144388 -0.000222 -0.001163" rpy="0 0 0"/>
       <inertia
-          ixx="0.01384106" ixy="0.00076195" ixz="-0.00011842"
-          iyy="0.12795959" iyz="0.00001926"
-          izz="0.13596145"/>
+          ixx="0.01219350" ixy="0.00078" ixz="-0.000112"
+          iyy="0.12351" iyz="0.00001833"
+          izz="0.13043"/>
     </inertial>
     <visual>

Commit message: [URDF]modified inertia of magnet airframe

File: robots/assemble_quadrotors/urdf/assemble_dual_quadrotors_female_mag.urdf.xacro (robot description, xacro)
@@ -115,10 +115,10 @@
       <!--     iyy="0.01398491" iyz="-0.00005390" -->
       <!--     izz="0.01819428"/> -->
-      <mass value = "1.247857" />
-      <origin xyz="-0.00279206 -0.00110497 0.00095251 " rpy="0 0 0"/>
+      <mass value = "1.23" />
+      <origin xyz="-0.00209 -0.00158 0.00106 " rpy="0 0 0"/>
       <inertia
-          ixx="0.00689482" ixy="0.00007765" ixz="-0.00038481"
-          iyy="0.01355710" iyz="-0.00005091"
-          izz="0.01760133"/>
+          ixx="0.00624" ixy="0.0000176" ixz="-0.000470"
+          iyy="0.0133" iyz="-0.0000457"
+          izz="0.0168"/>
     </inertial>
     <visual>

File: robots/assemble_quadrotors/urdf/assemble_dual_quadrotors_male_mag.urdf.xacro (robot description, xacro)
@@ -109,10 +109,10 @@
   <link name="main_body">
     <inertial>
-      <mass value = "1.26347288" />
-      <origin xyz="0.00295047 -0.00151693 0.00015592" rpy="0 0 0"/>
+      <mass value = "1.23" />
+      <origin xyz="0.00218 -0.00165 -0.00150" rpy="0 0 0"/>
     <inertia
-        ixx="0.00694153" ixy="0.00003221" ixz="-0.00070136"
-        iyy="0.01575032" iyz="-0.00003297"
-        izz="0.01974271"/>
+        ixx="0.00626" ixy="0.00002959" ixz="-0.000716"
+        iyy="0.0152" iyz="-0.00004101"
+        izz="0.0187"/>
     </inertial>
     <visual>

File: robots/assemble_quadrotors/urdf/assemble_dual_quadrotors_whole_female_mag.urdf.xacro (robot description, xacro)
@@ -109,10 +109,10 @@
   <link name="main_body">
     <inertial>
-      <mass value = "2.50834021" />
-      <origin xyz="-0.00140155 0.00021569 0.00055126" rpy="0 0 0"/>
+      <mass value = "2.46" />
+      <origin xyz="-0.00186 0.00003441 -0.00128" rpy="0 0 0"/>
       <inertia
-          ixx="0.01384106" ixy="0.00076195" ixz="0.00011842"
-          iyy="0.12795959" iyz="-0.00001926"
-          izz="0.13596145"/>
+          ixx="0.0125" ixy="0.000837" ixz="0.000138"
+          iyy="0.125" iyz="-0.00000554"
+          izz="0.132"/>
     </inertial>
     <visual>

File: robots/assemble_quadrotors/urdf/assemble_dual_quadrotors_whole_male_mag.urdf.xacro (robot description, xacro)
@@ -92,10 +92,10 @@
   <link name="root">
     <inertial>
-      <origin xyz="0 0 0" rpy="0 0 0"/>
-      <mass value="0.00001"/>
+      <mass value = "2.46" />
+      <origin xyz="0.00186 -0.00003441 -0.00128" rpy="0 0 0"/>
       <inertia
-          ixx="0.000001" ixy="0.0" ixz="0.0"
-          iyy="0.000001" iyz="0.0"
-          izz="0.000002"/>
+          ixx="0.0125" ixy="0.000837" ixz="-0.000138"
+          iyy="0.125" iyz="0.00000554"
+          izz="0.132"/>
     </inertial>
   </link>

Commit message: [URDF]modified urdf for battery

File: robots/assemble_quadrotors/urdf/assemble_dual_quadrotors_female_mag.urdf.xacro (robot description, xacro)
@@ -109,16 +109,10 @@
   <link name="main_body">
     <inertial>
-      <!-- <mass value = "1.427857" /> -->
-      <!-- <origin xyz="-0.00884209 -0.00096336 -0.00122007 " rpy="0 0 0"/> -->
-      <!-- <inertia -->
-      <!--     ixx="0.00716924" ixy="0.00006933" ixz="-0.00025713" -->
-      <!--     iyy="0.01398491" iyz="-0.00005390" -->
-      <!--     izz="0.01819428"/> -->
-      <mass value = "1.23" />
-      <origin xyz="-0.00209 -0.00158 0.00106 " rpy="0 0 0"/>
+      <mass value = "1.244" />
+      <origin xyz="-0.00452 -0.00138 0.0001977 " rpy="0 0 0"/>
       <inertia
-          ixx="0.00624" ixy="0.0000176" ixz="-0.000470"
-          iyy="0.0133" iyz="-0.0000457"
-          izz="0.0168"/>
+          ixx="0.00634" ixy="-0.0000162" ixz="-0.000522"
+          iyy="0.0146" iyz="-0.0000500"
+          izz="0.0183"/>
     </inertial>
     <visual>
@@ -137,7 +131,7 @@
   <!-- spinal -->
   <xacro:extra_module name = "fc" parent = "main_body" visible = "0" >
-    <origin xyz="0 0 0" rpy="0 0 0"/>
+    <origin xyz="-0.02 0 0" rpy="0 0 0"/>
     <inertial>
-      <mass value = "0.05" />
+      <mass value = "0.013" />
       <origin xyz="0 0 0" rpy="0 0 0"/>
       <inertia

File: robots/assemble_quadrotors/urdf/assemble_dual_quadrotors_male_mag.urdf.xacro (robot description, xacro)
@@ -109,10 +109,10 @@
   <link name="main_body">
     <inertial>
-      <mass value = "1.23" />
-      <origin xyz="0.00218 -0.00165 -0.00150" rpy="0 0 0"/>
+      <mass value = "1.2478" />
+      <origin xyz="-0.00246 -0.00144 -0.000238" rpy="0 0 0"/>
     <inertia
-        ixx="0.00626" ixy="0.00002959" ixz="-0.000716"
-        iyy="0.0152" iyz="-0.00004101"
-        izz="0.0187"/>
+        ixx="0.00636" ixy="-0.00000937" ixz="-0.000737"
+        iyy="0.0172" iyz="-0.0000451"
+        izz="0.0208"/>
     </inertial>
     <visual>
@@ -131,7 +131,7 @@
   <!-- spinal -->
   <xacro:extra_module name = "fc" parent = "main_body" visible = "0" >
-    <origin xyz="0 0 0" rpy="0 0 0"/>
+    <origin xyz="-0.02 0 0" rpy="0 0 0"/>
     <inertial>
-      <mass value = "0.05" />
+      <mass value = "0.013" />
       <origin xyz="0 0 0" rpy="0 0 0"/>
       <inertia

File: robots/assemble_quadrotors/urdf/assemble_dual_quadrotors_whole_female.urdf.xacro (robot description, xacro)
@@ -109,15 +109,13 @@
   <link name="main_body">
     <inertial>
-      <mass value = "2.5" />
-      <!-- <origin xyz="0.00401288 0.00002524 0.00751852" rpy="0 0 0"/> -->
-      <origin xyz="-0.01665965 0.00002872 0.00310773" rpy="0 0 0"/> <!-- for wierd -->
-      <!-- <origin xyz="0.0 0.0 0.0" rpy="0 0 0"/> -->
+      <mass value = "2.492" />
+      <origin xyz="-0.002 0.000 0.000" rpy="0 0 0"/>
       <inertia
-          ixx="0.01257219" ixy="0.00079619" ixz="0.00057445"
-          iyy="0.12647091" iyz="-0.00000082"
-          izz="0.13407114"/>
+          ixx="0.013" ixy="0.001" ixz="0.00"
+          iyy="0.133" iyz="0.000"
+          izz="0.14"/>
     </inertial>
     <visual>
-      <origin rpy="0 0 3.141592" xyz="0 0 0"/>
+      <origin rpy="0 0 0" xyz="0 0 0"/>
       <geometry>
         <mesh filename="package://assemble_quadrotors/urdf/mesh/Assemble_dual_quadrotors_v4.STL"/>
@@ -135,5 +133,5 @@
     <origin xyz="-0.22 0.0 0.0165" rpy="0 0 0"/>
     <inertial>
-      <mass value = "0.05" />
+      <mass value = "0.013" />
       <origin xyz="0 0 0" rpy="0 0 0"/>
       <inertia

File: robots/assemble_quadrotors/urdf/assemble_dual_quadrotors_whole_male_mag.urdf.xacro (robot description, xacro)
@@ -109,13 +109,13 @@
   <link name="main_body">
     <inertial>
-      <mass value = "2.50834021" />
-      <origin xyz="0.00140155 -0.00021569 0.00055126" rpy="0 0 0"/>
+      <mass value = "2.492" />
+      <origin xyz="0.002 0.000 0.000" rpy="0 0 0"/>
       <inertia
-          ixx="0.01384106" ixy="0.00076195" ixz="-0.00011842"
-          iyy="0.12795959" iyz="0.00001926"
-          izz="0.13596145"/>
+          ixx="0.013" ixy="0.001" ixz="0.00"
+          iyy="0.133" iyz="0.000"
+          izz="0.14"/>
     </inertial>
     <visual>
-      <origin rpy="0 0 3.141592" xyz="0 0 0"/>
+      <origin rpy="0 0 0" xyz="0 0 0"/>
       <geometry>
         <mesh filename="package://assemble_quadrotors/urdf/mesh/Assemble_dual_quadrotors_magnet_male.STL"/>
@@ -133,5 +133,5 @@
     <origin xyz="-0.22 0.0 0.0165" rpy="0 0 0"/>
     <inertial>
-      <mass value = "0.05" />
+      <mass value = "0.013" />
       <origin xyz="0 0 0" rpy="0 0 0"/>
       <inertia

Commit message: [URDF]modified unit urdf for battery

File: robots/assemble_quadrotors/urdf/assemble_dual_quadrotors_female_mag.urdf.xacro (robot description, xacro)
@@ -109,10 +109,10 @@
   <link name="main_body">
     <inertial>
-      <mass value = "1.244" />
-      <origin xyz="-0.00452 -0.00138 0.0001977 " rpy="0 0 0"/>
+      <mass value = "1.19" />
+      <origin xyz="0.008 -0.001 0.000044 " rpy="0 0 0"/>
       <inertia
-          ixx="0.00634" ixy="-0.0000162" ixz="-0.000522"
-          iyy="0.0146" iyz="-0.0000500"
-          izz="0.0183"/>
+          ixx="0.00635" ixy="-0.0000415" ixz="-0.000661"
+          iyy="0.0120" iyz="-0.0000605"
+          izz="0.0156"/>
     </inertial>
     <visual>

File: robots/assemble_quadrotors/urdf/assemble_dual_quadrotors_male_mag.urdf.xacro (robot description, xacro)
@@ -109,10 +109,10 @@
   <link name="main_body">
     <inertial>
-      <mass value = "1.2478" />
-      <origin xyz="-0.00246 -0.00144 -0.000238" rpy="0 0 0"/>
+      <mass value = "1.19" />
+      <origin xyz="0.00102 -0.00196 -0.000417" rpy="0 0 0"/>
     <inertia
-        ixx="0.00636" ixy="-0.00000937" ixz="-0.000737"
-        iyy="0.0172" iyz="-0.0000451"
-        izz="0.0208"/>
+        ixx="0.00636" ixy="0.0000666" ixz="-0.000868"
+        iyy="0.0142" iyz="-0.0000353"
+        izz="0.0177"/>
     </inertial>
     <visual>

Commit message: [Assembly] workaround to do aerial reconfiguration simulation

File: robots/assemble_quadrotors/urdf/assemble_dual_quadrotors_female_mag.urdf.xacro (robot description, xacro)
@@ -67,8 +67,8 @@
         <geometry>
           <xacro:if value="${direction == 1}">
-            <mesh filename="package://assemble_quadrotors/urdf/mesh/5_inchi_propeller.STL" />
+            <mesh filename="package://assemble_quadrotors/urdf/mesh/5inch_propeller.dae" />
           </xacro:if>
           <xacro:unless value="${direction == 1}">
-	    <mesh filename="package://assemble_quadrotors/urdf/mesh/5_inchi_propeller.STL" />
+	    <mesh filename="package://assemble_quadrotors/urdf/mesh/5inch_propeller.dae" />
           </xacro:unless>
         </geometry>
@@ -125,5 +125,5 @@
       <origin rpy="0 0 0" xyz="0 0 0"/>
       <geometry>
-        <mesh filename="package://assemble_quadrotors/urdf/mesh/Assemble_quadrotor_female_magnet.STL" />
+        <mesh filename="package://assemble_quadrotors/urdf/mesh/assemble_mag_femlae.dae" />
       </geometry>
     </visual>

File: robots/assemble_quadrotors/urdf/assemble_dual_quadrotors_male_mag.urdf.xacro (robot description, xacro)
@@ -67,8 +67,8 @@
         <geometry>
           <xacro:if value="${direction == 1}">
-            <mesh filename="package://assemble_quadrotors/urdf/mesh/5_inchi_propeller.STL" />
+            <mesh filename="package://assemble_quadrotors/urdf/mesh/5inch_propeller.dae" />
           </xacro:if>
           <xacro:unless value="${direction == 1}">
-	    <mesh filename="package://assemble_quadrotors/urdf/mesh/5_inchi_propeller.STL" />
+	    <mesh filename="package://assemble_quadrotors/urdf/mesh/5inch_propeller.dae" />
           </xacro:unless>
         </geometry>
@@ -119,5 +119,5 @@
       <origin rpy="0 0 0" xyz="0 0 0"/>
       <geometry>
-        <mesh filename="package://assemble_quadrotors/urdf/mesh/Assemble_quadrotor_male_magnet.STL"/>
+        <mesh filename="package://assemble_quadrotors/urdf/mesh/assemble_mag_male.dae"/>
       </geometry>
     </visual>
@@ -155,9 +155,9 @@
           iyy="0.0001" iyz="0.0000" izz="0.0001"/>
     </inertial>
-    <visual>
-      <geometry>
-        <box size="0.04 0.04 0.04"/>
-      </geometry>
-    </visual>
+    <!-- <visual> -->
+    <!--   <geometry> -->
+    <!--     <box size="0.04 0.04 0.04"/> -->
+    <!--   </geometry> -->
+    <!-- </visual> -->
   </link>
   <joint name="base_dummy_arm_joint" type="fixed">
@@ -211,10 +211,10 @@
       </geometry>
     </collision>
-    <visual>
-      <origin xyz="0 0 0" rpy="0.0 0 0"/>
-      <geometry>
-        <box size="0.04 0.04 0.04"/>
-      </geometry>
-    </visual>
+    <!-- <visual> -->
+    <!--   <origin xyz="0 0 0" rpy="0.0 0 0"/> -->
+    <!--   <geometry> -->
+    <!--     <box size="0.04 0.04 0.04"/> -->
+    <!--   </geometry> -->
+    <!-- </visual> -->
   </link>
   <transmission name="joint_tran1">
