Commit message: [URDF][Trirotor] modified urdf and servo yaml in order to adjust ot trirotor

File: robots/gimbalrotor/robots/gimbalrotor.urdf.xacro (robot description, xacro)
@@ -4,8 +4,7 @@
   <xacro:include filename="$(find gimbalrotor)/urdf/gimbalrotor.urdf.xacro" />
   <xacro:include filename="$(find gimbalrotor)/urdf/common.xacro" />
-  <xacro:gimbalrotor_center_link child1="1" child2="2" child3="3" child4="4"/>
+  <xacro:gimbalrotor_center_link child1="1" child2="2" child3="3"/>
   <xacro:gimbalrotor_thrust_link self="1" rotor_direction="1"/>
   <xacro:gimbalrotor_thrust_link self="2" rotor_direction="-1"/>
   <xacro:gimbalrotor_thrust_link self="3" rotor_direction="1"/>
-  <xacro:gimbalrotor_thrust_link self="4" rotor_direction="-1"/>
 </robot>

File: robots/gimbalrotor/urdf/gimbalrotor.urdf.xacro (robot description, xacro)
@@ -2,5 +2,5 @@
 <robot
     xmlns:xacro="http://www.ros.org/wiki/xacro" name="gimbalrotor_link" >
-  <xacro:macro name="gimbalrotor_center_link" params="child1 child2 child3 child4">
+  <xacro:macro name="gimbalrotor_center_link" params="child1 child2 child3">
     ## dummy
     <link name="root">
@@ -23,14 +23,14 @@
     <link name="base_link">
       <inertial>
-        <origin xyz="0.0 0.0 0.0165" rpy="0 0 0"/>
-        <mass value="0.1753"/>
-        <inertia
-            ixx="0.0004" iyy="0.0004" izz="0.0008"
+        <origin xyz="-0.082255 0.000157 0.014372" rpy="0 0 0"/>
+        <mass value="1.076"/>
+        <inertia
+            ixx="0.005338" iyy="0.006510" izz="0.01052"
             ixy="0.00000" ixz="0.0000" iyz="0.00000"/>
       </inertial>
       <visual>
-        <origin xyz="0 0 -0.0165" rpy="0 0 0"/>
-        <geometry>
-          <mesh filename="package://gimbalrotor/urdf/mesh/base_link.STL"/>
+        <origin xyz="0 0 0" rpy="0 0 0"/>
+        <geometry>
+          <mesh filename="package://gimbalrotor/urdf/mesh/trirotor_base_link.dae" scale="0.001 0.001 0.001"/>
         </geometry>
       </visual>
@@ -38,5 +38,5 @@
         <origin xyz="0 0 0" rpy="0 0 0"/>
         <geometry>
-          <box size="0.25 0.25 0.035"/>
+          <box size="0.234 0.3 0.1"/>
         </geometry>
       </collision>
@@ -59,115 +59,51 @@
       <axis xyz="0 0 1"/>
     </joint>
-    ## rotor arms
+    ## dummy rotor arms
     <link name="rotor_arm${child1}">
       <inertial>
-        <origin xyz="0.0486 0 0.0161" rpy="0 0 0"/>
-        <mass value="0.088"/>
-        <inertia
-            ixx="0.000001" ixy="0.0" ixz="0.0"
-            iyy="0.0001" iyz="0.0"
-            izz="0.0001"/>
-      </inertial>
-      <visual>
-        <origin xyz="0 0 0" rpy="0 0 0"/>
-        <geometry>
-          <mesh filename="package://gimbalrotor/urdf/mesh/rotor_arm.STL"/>
-        </geometry>
-      </visual>
-      <collision>
-        <origin xyz="0 0 0" rpy="0 0 0"/>
-        <geometry>
-          <box size="0.131 0.0325 0.065"/>
-        </geometry>
-      </collision>
+        <origin xyz="0 0 0" rpy="0 0 0"/>
+        <mass value="0.001"/>
+        <inertia
+            ixx="0.000001" ixy="0.0" ixz="0.0"
+            iyy="0.000001" iyz="0.0"
+            izz="0.000001"/>
+      </inertial>
     </link>
     <joint name="base_arm_joint${child1}" type="fixed">
       <parent link="base_link"/>
       <child link="rotor_arm${child1}"/>
-      <origin rpy="0 0 ${pi/4}" xyz="0.051 0.051 0.0"/>
+      <origin rpy="0 0 ${-pi/2}" xyz="0 -0.154 0.051"/>
       <axis xyz="0 0 1"/>
     </joint>
     <link name="rotor_arm${child2}">
       <inertial>
-        <origin xyz="0.0486 0 0.0161" rpy="0 0 0"/>
-        <mass value="0.088"/>
-        <inertia
-            ixx="0.000001" ixy="0.0" ixz="0.0"
-            iyy="0.0001" iyz="0.0"
-            izz="0.0001"/>
-      </inertial>
-      <visual>
-        <origin xyz="0 0 0" rpy="0 0 0"/>
-        <geometry>
-          <mesh filename="package://gimbalrotor/urdf/mesh/rotor_arm.STL"/>
-        </geometry>
-      </visual>
-      <collision>
-        <origin xyz="0 0 0" rpy="0 0 0"/>
-        <geometry>
-          <box size="0.131 0.0325 0.065"/>
-        </geometry>p
-      </collision>
+        <origin xyz="0 0 0" rpy="0 0 0"/>
+        <mass value="0.0001"/>
+        <inertia
+            ixx="0.000001" ixy="0.0" ixz="0.0"
+            iyy="0.000001" iyz="0.0"
+            izz="0.000001"/>
+      </inertial>
     </link>
     <joint name="base_arm_joint${child2}" type="fixed">
       <parent link="base_link"/>
       <child link="rotor_arm${child2}"/>
-      <origin rpy="0 0 ${pi*3.0/4.0}" xyz="-0.051 0.051 0.0"/>
+      <origin rpy="0 0 ${pi/2}" xyz="0 0.154 0.051"/>
       <axis xyz="0 0 1"/>
     </joint>
     <link name="rotor_arm${child3}">
       <inertial>
-        <origin xyz="0.0486 0 0.0161" rpy="0 0 0"/>
-        <mass value="0.088"/>
-        <inertia
-            ixx="0.000001" ixy="0.0" ixz="0.0"
-            iyy="0.0001" iyz="0.0"
-            izz="0.0001"/>
-      </inertial>
-      <visual>
-        <origin xyz="0 0 0" rpy="0 0 0"/>
-        <geometry>
-          <mesh filename="package://gimbalrotor/urdf/mesh/rotor_arm.STL"/>
-        </geometry>
-      </visual>
-      <collision>
-        <origin xyz="0 0 0" rpy="0 0 0"/>
-        <geometry>
-          <box size="0.131 0.0325 0.065"/>
-        </geometry>
-      </collision>
+        <origin xyz="0 0 0" rpy="0 0 0"/>
+        <mass value="0.0001"/>
+        <inertia
+            ixx="0.000001" ixy="0.0" ixz="0.0"
+            iyy="0.000001" iyz="0.0"
+            izz="0.000001"/>
+      </inertial>
     </link>
     <joint name="base_arm_joint${child3}" type="fixed">
       <parent link="base_link"/>
       <child link="rotor_arm${child3}"/>
-      <origin rpy="0 0 ${pi*5.0/4.0}" xyz="-0.051 -0.051 0.0"/>
-      <axis xyz="0 0 1"/>
-    </joint>
-    <link name="rotor_arm${child4}">
-      <inertial>
-        <origin xyz="0.0486 0 0.0161" rpy="0 0 0"/>
-        <mass value="0.088"/>
-        <inertia
-            ixx="0.000001" ixy="0.0" ixz="0.0"
-            iyy="0.0001" iyz="0.0"
-            izz="0.0001"/>
-      </inertial>
-      <visual>
-        <origin xyz="0 0 0" rpy="0 0 0"/>
-        <geometry>
-          <mesh filename="package://gimbalrotor/urdf/mesh/rotor_arm.STL"/>
-        </geometry>
-      </visual>
-      <collision>
-        <origin xyz="0 0 0" rpy="0 0 0"/>
-        <geometry>
-          <box size="0.131 0.0325 0.065"/>
-        </geometry>
-      </collision>
-    </link>
-    <joint name="base_arm_joint${child4}" type="fixed">
-      <parent link="base_link"/>
-      <child link="rotor_arm${child4}"/>
-      <origin rpy="0 0 ${-pi/4.0}" xyz="0.051 -0.051 0.0"/>
+      <origin rpy="0 0 ${pi}" xyz="-0.214 0 0.051"/>
       <axis xyz="0 0 1"/>
     </joint>
@@ -179,20 +115,20 @@
     <link name="gimbal_link${self}">
       <inertial>
-        <origin xyz="0.018 0.00 0.00438" rpy="0 0 0"/>
-        <mass value="0.1095"/>
-        <inertia
-            ixx="0.00002989" iyy="0.00002848" izz="0.0002698"
+        <origin xyz="0.076255 0 0" rpy="0 0 0"/>
+        <mass value="0.148"/>
+        <inertia
+            ixx="0.000299" iyy="0.000157" izz="0.000386"
             ixy="0.0000" ixz="-0.0000" iyz="0.00000"/>
       </inertial>
       <collision>
-        <origin xyz="0.0 0 0" rpy="0 0 0"/>
-        <geometry>
-          <cylinder radius="0.018" length="0.033"/>
+        <origin xyz="0.076255 0 0" rpy="0 0 0"/>
+        <geometry>
+          <cylinder radius="0.1" length="0.1"/>
         </geometry>
       </collision>
       <visual>
-        <origin xyz="0 0 0" rpy="0 0 0"/>
-        <geometry>
-          <mesh filename="package://gimbalrotor/urdf/mesh/rotor_module.STL"/>
+        <origin xyz="0 0 0" rpy="0 0 ${-pi/2}"/>
+        <geometry>
+          <mesh filename="package://gimbalrotor/urdf/mesh/thrust_link_left_straight.dae" scale="0.001 0.001 0.001"/>
         </geometry>
       </visual>
@@ -228,5 +164,5 @@
       <parent link="rotor_arm${self}"/>
       <child link="gimbal_link${self}"/>
-      <origin rpy="0 0 0" xyz="0.077 0 0.0385"/>
+      <origin rpy="0 0 0" xyz="0 0 0"/>
       <axis xyz="1 0 0"/>
       <dynamics damping="0.8" friction="0.0"/>
@@ -246,5 +182,5 @@
       <parent link="gimbal_link${self}"/>
       <child link="rotor_parent${self}"/>
-      <origin rpy="0 0 0" xyz="0.018 0.00 0.00438"/>
+      <origin rpy="0 0 0" xyz="0.0835 0 0"/>
       <axis xyz="0 0 ${rotor_direction}"/>
     </joint>

Commit message: [WIP][Gimbalrotor] modified urdf for ant module

File: robots/gimbalrotor/robots/gimbalrotor.urdf.xacro (robot description, xacro)
@@ -68,5 +68,5 @@
     <parent link="dummy_palm"/>
     <child link="dummy_gripper"/>
-    <origin xyz="0.05 0 0" rpy="0 0 0"/>
+    <origin xyz="0.04 0 0" rpy="0 0 0"/>
     <axis xyz="1 0 0"/>
     <limit lower="0" upper="0" effort="0" velocity="0"/>
@@ -81,14 +81,8 @@
           iyy="0.0001" iyz="0.0000" izz="0.0001"/>
     </inertial>
-    <visual>
-      <origin xyz="0.0 0 0" rpy="0.0 0 0"/>
-      <geometry>
-        <box size="0.1 0.05 0.05"/>
-      </geometry>
-    </visual>
     <collision>
       <origin xyz="0.0 0 0" rpy="0 0 0"/>
       <geometry>
-        <box size="0.1 0.05 0.05"/>
+        <box size="0.06 0.05 0.05"/>
       </geometry>
       <material name="red">

File: robots/gimbalrotor/urdf/gimbalrotor.urdf.xacro (robot description, xacro)
@@ -32,5 +32,5 @@
         <origin xyz="0 0 -0.0165" rpy="0 0 0"/>
         <geometry>
-          <mesh filename="package://gimbalrotor/urdf/mesh/base_link.STL"/>
+          <mesh filename="package://gimbalrotor/urdf/mesh/ants_module_base.STL"/>
         </geometry>
       </visual>
@@ -38,5 +38,5 @@
         <origin xyz="0 0 0" rpy="0 0 0"/>
         <geometry>
-          <box size="0.25 0.25 0.035"/>
+          <box size="0.5 0.5 0.15"/>
         </geometry>
       </collision>
@@ -59,115 +59,67 @@
       <axis xyz="0 0 1"/>
     </joint>
-    ## rotor arms
+    ## dummy rotor arms
     <link name="rotor_arm${child1}">
       <inertial>
+        <origin xyz="0 0 0" rpy="0 0 0"/>
+        <mass value="0.0001"/>
+        <inertia
+            ixx="0.000001" ixy="0.0" ixz="0.0"
+            iyy="0.0001" iyz="0.0"
+            izz="0.0001"/>
+      </inertial>
+    </link>
+    <joint name="base_arm_joint${child1}" type="fixed">
+      <parent link="base_link"/>
+      <child link="rotor_arm${child1}"/>
+      <origin rpy="0 0 ${pi/4}" xyz="0.124 0.124 0.0555"/>
+      <axis xyz="0 0 1"/>
+    </joint>
+    <link name="rotor_arm${child2}">
+      <inertial>
         <origin xyz="0.0486 0 0.0161" rpy="0 0 0"/>
-        <mass value="0.088"/>
-        <inertia
-            ixx="0.000001" ixy="0.0" ixz="0.0"
-            iyy="0.0001" iyz="0.0"
-            izz="0.0001"/>
-      </inertial>
-      <visual>
-        <origin xyz="0 0 0" rpy="0 0 0"/>
-        <geometry>
-          <mesh filename="package://gimbalrotor/urdf/mesh/rotor_arm.STL"/>
-        </geometry>
-      </visual>
-      <collision>
-        <origin xyz="0 0 0" rpy="0 0 0"/>
-        <geometry>
-          <box size="0.131 0.0325 0.065"/>
-        </geometry>
-      </collision>
-    </link>
-    <joint name="base_arm_joint${child1}" type="fixed">
-      <parent link="base_link"/>
-      <child link="rotor_arm${child1}"/>
-      <origin rpy="0 0 ${pi/4}" xyz="0.051 0.051 0.0"/>
-      <axis xyz="0 0 1"/>
-    </joint>
-    <link name="rotor_arm${child2}">
+        <mass value="0.0001"/>
+        <inertia
+            ixx="0.000001" ixy="0.0" ixz="0.0"
+            iyy="0.0001" iyz="0.0"
+            izz="0.0001"/>
+      </inertial>
+    </link>
+    <joint name="base_arm_joint${child2}" type="fixed">
+      <parent link="base_link"/>
+      <child link="rotor_arm${child2}"/>
+      <origin rpy="0 0 ${pi*3.0/4.0}" xyz="-0.124 0.124 0.0555"/>
+      <axis xyz="0 0 1"/>
+    </joint>
+    <link name="rotor_arm${child3}">
       <inertial>
         <origin xyz="0.0486 0 0.0161" rpy="0 0 0"/>
-        <mass value="0.088"/>
-        <inertia
-            ixx="0.000001" ixy="0.0" ixz="0.0"
-            iyy="0.0001" iyz="0.0"
-            izz="0.0001"/>
-      </inertial>
-      <visual>
-        <origin xyz="0 0 0" rpy="0 0 0"/>
-        <geometry>
-          <mesh filename="package://gimbalrotor/urdf/mesh/rotor_arm.STL"/>
-        </geometry>
-      </visual>
-      <collision>
-        <origin xyz="0 0 0" rpy="0 0 0"/>
-        <geometry>
-          <box size="0.131 0.0325 0.065"/>
-        </geometry>p
-      </collision>
-    </link>
-    <joint name="base_arm_joint${child2}" type="fixed">
-      <parent link="base_link"/>
-      <child link="rotor_arm${child2}"/>
-      <origin rpy="0 0 ${pi*3.0/4.0}" xyz="-0.051 0.051 0.0"/>
-      <axis xyz="0 0 1"/>
-    </joint>
-    <link name="rotor_arm${child3}">
+        <mass value="0.0001"/>
+        <inertia
+            ixx="0.000001" ixy="0.0" ixz="0.0"
+            iyy="0.0001" iyz="0.0"
+            izz="0.0001"/>
+      </inertial>
+    </link>
+    <joint name="base_arm_joint${child3}" type="fixed">
+      <parent link="base_link"/>
+      <child link="rotor_arm${child3}"/>
+      <origin rpy="0 0 ${pi*5.0/4.0}" xyz="-0.124 -0.124 0.0555"/>
+      <axis xyz="0 0 1"/>
+    </joint>
+    <link name="rotor_arm${child4}">
       <inertial>
         <origin xyz="0.0486 0 0.0161" rpy="0 0 0"/>
-        <mass value="0.088"/>
-        <inertia
-            ixx="0.000001" ixy="0.0" ixz="0.0"
-            iyy="0.0001" iyz="0.0"
-            izz="0.0001"/>
-      </inertial>
-      <visual>
-        <origin xyz="0 0 0" rpy="0 0 0"/>
-        <geometry>
-          <mesh filename="package://gimbalrotor/urdf/mesh/rotor_arm.STL"/>
-        </geometry>
-      </visual>
-      <collision>
-        <origin xyz="0 0 0" rpy="0 0 0"/>
-        <geometry>
-          <box size="0.131 0.0325 0.065"/>
-        </geometry>
-      </collision>
-    </link>
-    <joint name="base_arm_joint${child3}" type="fixed">
-      <parent link="base_link"/>
-      <child link="rotor_arm${child3}"/>
-      <origin rpy="0 0 ${pi*5.0/4.0}" xyz="-0.051 -0.051 0.0"/>
-      <axis xyz="0 0 1"/>
-    </joint>
-    <link name="rotor_arm${child4}">
-      <inertial>
-        <origin xyz="0.0486 0 0.0161" rpy="0 0 0"/>
-        <mass value="0.088"/>
-        <inertia
-            ixx="0.000001" ixy="0.0" ixz="0.0"
-            iyy="0.0001" iyz="0.0"
-            izz="0.0001"/>
-      </inertial>
-      <visual>
-        <origin xyz="0 0 0" rpy="0 0 0"/>
-        <geometry>
-          <mesh filename="package://gimbalrotor/urdf/mesh/rotor_arm.STL"/>
-        </geometry>
-      </visual>
-      <collision>
-        <origin xyz="0 0 0" rpy="0 0 0"/>
-        <geometry>
-          <box size="0.131 0.0325 0.065"/>
-        </geometry>
-      </collision>
+        <mass value="0.0001"/>
+        <inertia
+            ixx="0.000001" ixy="0.0" ixz="0.0"
+            iyy="0.0001" iyz="0.0"
+            izz="0.0001"/>
+      </inertial>
     </link>
     <joint name="base_arm_joint${child4}" type="fixed">
       <parent link="base_link"/>
       <child link="rotor_arm${child4}"/>
-      <origin rpy="0 0 ${-pi/4.0}" xyz="0.051 -0.051 0.0"/>
+      <origin rpy="0 0 ${-pi/4.0}" xyz="0.124 -0.124 0.0555"/>
       <axis xyz="0 0 1"/>
     </joint>
@@ -228,5 +180,5 @@
       <parent link="rotor_arm${self}"/>
       <child link="gimbal_link${self}"/>
-      <origin rpy="0 0 0" xyz="0.077 0 0.0385"/>
+      <origin rpy="0 0 0" xyz="0 0 0"/>
       <axis xyz="1 0 0"/>
       <dynamics damping="0.8" friction="0.0"/>
