Commit message: [Ants][temp]unko

File: robots/gimbalrotor/robots/quad/gimbalrotor.gazebo.xacro (robot description, xacro)
@@ -8,19 +8,19 @@
   <xacro:gazebo_spinal robot_name="$(arg robot_name)" mag_frame="fc" />
   <!-- gazebo plugin for docking mech -->
-  <gazebo>
-    <plugin name="gazebo_grasp_fix" filename="libgazebo_grasp_fix.so">
-      <arm>
-        <arm_name>docking_mech</arm_name>
-        <palm_link>dummy_palm</palm_link>
-        <gripper_link>dummy_gripper</gripper_link>
-      </arm>
-      <forces_angle_tolerance>90</forces_angle_tolerance>
-      <update_rate>50</update_rate>
-      <grip_count_threshold>0</grip_count_threshold>
-      <max_grip_count>1</max_grip_count>
-      <release_tolerance>1</release_tolerance>
-      <disable_collisions_on_attach>false</disable_collisions_on_attach>
-      <contact_topic>__default_topic__</contact_topic>
-    </plugin>
-  </gazebo>
+  <!-- <gazebo> -->
+  <!--   <plugin name="gazebo_grasp_fix" filename="libgazebo_grasp_fix.so"> -->
+  <!--     <arm> -->
+  <!--       <arm_name>docking_mech</arm_name> -->
+  <!--       <palm_link>dummy_palm</palm_link> -->
+  <!--       <gripper_link>dummy_gripper</gripper_link> -->
+  <!--     </arm> -->
+  <!--     <forces_angle_tolerance>90</forces_angle_tolerance> -->
+  <!--     <update_rate>50</update_rate> -->
+  <!--     <grip_count_threshold>0</grip_count_threshold> -->
+  <!--     <max_grip_count>1</max_grip_count> -->
+  <!--     <release_tolerance>1</release_tolerance> -->
+  <!--     <disable_collisions_on_attach>false</disable_collisions_on_attach> -->
+  <!--     <contact_topic>__default_topic__</contact_topic> -->
+  <!--   </plugin> -->
+  <!-- </gazebo> -->
 </robot>

File: robots/gimbalrotor/robots/quad/gimbalrotor.urdf.xacro (robot description, xacro)
@@ -9,70 +9,73 @@
   <xacro:gimbalrotor_thrust_link self="3" rotor_direction="1"/>
   <xacro:gimbalrotor_thrust_link self="4" rotor_direction="-1"/>
-  ##### dummy grasp links ####
-  <joint name="base_dummy_arm_joint" type="fixed">
-    <parent link="base_link"/>
-    <child link="dummy_arm"/>
-    <origin xyz="0.22 0 0.1455" rpy="0 0 0"/>
-  </joint>
-  <link name="dummy_arm">
-    <inertial>
-      <mass value = "0.01" />
-      <origin xyz="0.05 0 0" rpy="0 0 0"/>
-      <inertia
-          ixx="0.0001" ixy="0.0000" ixz="0.0000"
-          iyy="0.0001" iyz="0.0000" izz="0.0001"/>
-    </inertial>
-  </link>
-  <joint name="dummy_arm_palm_joint" type="revolute">
-    <parent link="dummy_arm"/>
-    <child link="dummy_palm"/>
-    <origin xyz="0.02 0 0" rpy="0 0 0"/>
-    <axis xyz="1 0 0"/>
-    <limit lower="0" upper="0" effort="0" velocity="0"/>
-    <dynamics damping="0.2" friction="0.02"/>
-  </joint>
-  <link name="dummy_palm">
-    <inertial>
-      <mass value = "0.001" />
-      <origin xyz="0 0 0" rpy="0 0 0"/>
-      <inertia
-          ixx="0.0001" ixy="0.0000" ixz="0.0000"
-          iyy="0.0001" iyz="0.0000" izz="0.0001"/>
-    </inertial>
-    <collision>
-      <origin xyz="0 0 0" rpy="0 0 0"/>
-      <geometry>
-        <box size="0.04 0.04 0.04"/>
-      </geometry>
-    </collision>
-  </link>
-  <joint name="dummy_palm_gripper_joint" type="revolute">
-    <parent link="dummy_palm"/>
-    <child link="dummy_gripper"/>
-    <origin xyz="0 0 0" rpy="0 0 0"/>
-    <axis xyz="1 0 0"/>
-    <limit lower="0" upper="0" effort="0" velocity="0"/>
-    <dynamics damping="0.2" friction="0.02"/>
-  </joint>
-  <link name="dummy_gripper">
-    <inertial>
-      <mass value = "0.001" />
-      <origin xyz="0.0 0 0" rpy="0 0 0"/>
-      <inertia
-          ixx="0.0001" ixy="0.0000" ixz="0.0000"
-          iyy="0.0001" iyz="0.0000" izz="0.0001"/>
-    </inertial>
-    <collision>
-      <origin xyz="0 0 0" rpy="0 0 0"/>
-      <geometry>
-        <box size="0.04 0.04 0.04"/>
-      </geometry>
-    </collision>
-    <visual>
-      <origin xyz="0 0 0" rpy="0.0 0 0"/>
-      <geometry>
-        <box size="0.04 0.04 0.04"/>
-      </geometry>
-    </visual>
-  </link>
+  <!-- ##### dummy grasp links #### -->
+  <!-- <joint name="base_dummy_arm_joint" type="fixed"> -->
+  <!--   <parent link="base_link"/> -->
+  <!--   <child link="dummy_arm"/> -->
+  <!--   <origin xyz="0.22 0 0.1455" rpy="0 0 0"/> -->
+  <!-- </joint> -->
+  <!-- <link name="dummy_arm"> -->
+  <!--   <inertial> -->
+  <!--     <origin xyz="0 0 0" rpy="0 0 0"/> -->
+  <!--     <mass value="0.0001"/> -->
+  <!--     <inertia -->
+  <!--         ixx="0.000001" ixy="0.0" ixz="0.0" -->
+  <!--         iyy="0.0001" iyz="0.0" -->
+  <!--         izz="0.0001"/> -->
+  <!--   </inertial> -->
+  <!-- </link> -->
+  <!-- <joint name="dummy_arm_palm_joint" type="revolute"> -->
+  <!--   <parent link="dummy_arm"/> -->
+  <!--   <child link="dummy_palm"/> -->
+  <!--   <origin xyz="0.02 0 0" rpy="0 0 0"/> -->
+  <!--   <axis xyz="0 0 1"/> -->
+  <!--   <limit lower="0" upper="0" effort="0" velocity="0"/> -->
+  <!--   <dynamics damping="0.2" friction="0.02"/> -->
+  <!-- </joint> -->
+  <!-- <link name="dummy_palm"> -->
+  <!--   <inertial> -->
+  <!--     <origin xyz="0 0 0" rpy="0 0 0"/> -->
+  <!--     <mass value="0.0001"/> -->
+  <!--     <inertia -->
+  <!--         ixx="0.000001" ixy="0.0" ixz="0.0" -->
+  <!--         iyy="0.0001" iyz="0.0" -->
+  <!--         izz="0.0001"/> -->
+  <!--   </inertial> -->
+  <!--   <collision> -->
+  <!--     <origin xyz="0 0 0" rpy="0 0 0"/> -->
+  <!--     <geometry> -->
+  <!--       <box size="0.04 0.04 0.04"/> -->
+  <!--     </geometry> -->
+  <!--   </collision> -->
+  <!-- </link> -->
+  <!-- <joint name="dummy_palm_gripper_joint" type="revolute"> -->
+  <!--   <parent link="dummy_palm"/> -->
+  <!--   <child link="dummy_gripper"/> -->
+  <!--   <origin xyz="0 0 0" rpy="0 0 0"/> -->
+  <!--   <axis xyz="0 0 1"/> -->
+  <!--   <limit lower="0" upper="0" effort="0" velocity="0"/> -->
+  <!--   <dynamics damping="0.2" friction="0.02"/> -->
+  <!-- </joint> -->
+  <!-- <link name="dummy_gripper"> -->
+  <!--   <inertial> -->
+  <!--     <origin xyz="0 0 0" rpy="0 0 0"/> -->
+  <!--     <mass value="0.0001"/> -->
+  <!--     <inertia -->
+  <!--         ixx="0.000001" ixy="0.0" ixz="0.0" -->
+  <!--         iyy="0.0001" iyz="0.0" -->
+  <!--         izz="0.0001"/> -->
+  <!--   </inertial> -->
+  <!--   <collision> -->
+  <!--     <origin xyz="0 0 0" rpy="0 0 0"/> -->
+  <!--     <geometry> -->
+  <!--       <box size="0.04 0.04 0.04"/> -->
+  <!--     </geometry> -->
+  <!--   </collision> -->
+  <!--   <visual> -->
+  <!--     <origin xyz="0 0 0" rpy="0.0 0 0"/> -->
+  <!--     <geometry> -->
+  <!--       <box size="0.04 0.04 0.04"/> -->
+  <!--     </geometry> -->
+  <!--   </visual> -->
+  <!-- </link> -->
 </robot>

File: robots/gimbalrotor/urdf/quad/gimbalrotor.urdf.xacro (robot description, xacro)
@@ -7,9 +7,9 @@
       <inertial>
         <origin xyz="0 0 0" rpy="0 0 0"/>
-        <mass value="0.00001"/>
-        <inertia
-            ixx="0.000001" ixy="0.0" ixz="0.0"
-            iyy="0.000001" iyz="0.0"
-            izz="0.000001"/>
+        <mass value="0.0001"/>
+        <inertia
+            ixx="0.0001" ixy="0.0" ixz="0.0"
+            iyy="0.0001" iyz="0.0"
+            izz="0.0002"/>
       </inertial>
     </link>
@@ -26,9 +26,9 @@
         <mass value="1.82"/>
         <inertia
-            ixx="0.0511797" iyy="0.0835848" izz="0.1010814"
-            ixy="-0.0000001" ixz="-0.0015934" iyz="0.0000027"/>
+            ixx="0.05" iyy="0.08" izz="0.10"
+            ixy="0.0" ixz="0.0" iyz="0.0"/>
       </inertial>
       <visual>
-        <origin xyz="0 0 0" rpy="0 0 0"/>
+        <origin xyz="0 0 0" rpy="0 0 3.141592"/>
         <geometry>
           <mesh filename="package://gimbalrotor/urdf/quad/mesh/base_link.dae"/>
@@ -46,9 +46,9 @@
       <inertial>
         <origin xyz="0 0 0" rpy="0 0 0"/>
-        <mass value="0.00001"/>
-        <inertia
-            ixx="0.000001" ixy="0.0" ixz="0.0"
-            iyy="0.000001" iyz="0.0"
-            izz="0.000001"/>
+        <mass value="0.0001"/>
+        <inertia
+            ixx="0.0001" ixy="0.0" ixz="0.0"
+            iyy="0.0001" iyz="0.0"
+            izz="0.0002"/>
       </inertial>
     </link>
@@ -63,9 +63,9 @@
       <inertial>
         <origin xyz="0 0 0" rpy="0 0 0"/>
-        <mass value="0.0001"/>
-        <inertia
-            ixx="0.000001" ixy="0.0" ixz="0.0"
-            iyy="0.0001" iyz="0.0"
-            izz="0.0001"/>
+        <mass value="0.1"/>
+        <inertia
+            ixx="0.001" ixy="0.0" ixz="0.0"
+            iyy="0.001" iyz="0.0"
+            izz="0.002"/>
       </inertial>
     </link>
@@ -78,10 +78,10 @@
     <link name="rotor_arm${child2}">
       <inertial>
-        <origin xyz="0.0486 0 0.0161" rpy="0 0 0"/>
-        <mass value="0.0001"/>
-        <inertia
-            ixx="0.000001" ixy="0.0" ixz="0.0"
-            iyy="0.0001" iyz="0.0"
-            izz="0.0001"/>
+        <origin xyz="0 0 0" rpy="0 0 0"/>
+        <mass value="0.1"/>
+        <inertia
+            ixx="0.001" ixy="0.0" ixz="0.0"
+            iyy="0.001" iyz="0.0"
+            izz="0.002"/>
       </inertial>
     </link>
@@ -94,10 +94,10 @@
     <link name="rotor_arm${child3}">
       <inertial>
-        <origin xyz="0.0486 0 0.0161" rpy="0 0 0"/>
-        <mass value="0.0001"/>
-        <inertia
-            ixx="0.000001" ixy="0.0" ixz="0.0"
-            iyy="0.0001" iyz="0.0"
-            izz="0.0001"/>
+        <origin xyz="0 0 0" rpy="0 0 0"/>
+        <mass value="0.1"/>
+        <inertia
+            ixx="0.001" ixy="0.0" ixz="0.0"
+            iyy="0.001" iyz="0.0"
+            izz="0.002"/>
       </inertial>
     </link>
@@ -110,10 +110,10 @@
     <link name="rotor_arm${child4}">
       <inertial>
-        <origin xyz="0.0486 0 0.0161" rpy="0 0 0"/>
-        <mass value="0.0001"/>
-        <inertia
-            ixx="0.000001" ixy="0.0" ixz="0.0"
-            iyy="0.0001" iyz="0.0"
-            izz="0.0001"/>
+        <origin xyz="0 0 0" rpy="0 0 0"/>
+        <mass value="0.1"/>
+        <inertia
+            ixx="0.001" ixy="0.0" ixz="0.0"
+            iyy="0.001" iyz="0.0"
+            izz="0.002"/>
       </inertial>
     </link>
@@ -134,6 +134,6 @@
         <mass value="0.1333"/>
         <inertia
-            ixx="0.00005310" iyy="0.00005269" izz="0.00005333"
-            ixy="-0.00000001" ixz="0.00000064" iyz="0.00000"/>
+            ixx="0.0005" iyy="0.0005" izz="0.0005"
+            ixy="0" ixz="0" iyz="0.0"/>
       </inertial>
       <collision>
@@ -151,24 +151,13 @@
     </link>
     <xacro:damping_factor link="gimbal_link${self}"/>
-    ## rotor parent link (virtual)
-    <link name="rotor_parent${self}">
-      <inertial>
-        <origin xyz="0 0 0" rpy="0 0 0"/>
-        <mass value="0.00001"/>
-        <inertia
-            ixx="0.000001" ixy="0.0" ixz="0.0"
-            iyy="0.000001" iyz="0.0"
-            izz="0.000001"/>
-      </inertial>
-    </link>
     ## thrust link (virtual)
     <link name="thrust${self}">
       <inertial>
         <origin xyz="0 0 0" rpy="0 0 0"/>
-        <mass value="0.00001"/>
-        <inertia
-            ixx="0.001" ixy="0.0" ixz="0.0"
-            iyy="0.001" iyz="0.0"
-            izz="0.001"/>
+        <mass value="0.01"/>
+        <inertia
+            ixx="0.001" ixy="0.0" ixz="0.0"
+            iyy="0.001" iyz="0.0"
+            izz="0.002"/>
       </inertial>
     </link>
@@ -194,17 +183,10 @@
       </actuator>
     </transmission>
-    #### rotor parent link joint (virtual) ####
-    <joint name="rotor_parent_link_joint${self}" type="fixed">
-      <parent link="gimbal_link${self}"/>
-      <child link="rotor_parent${self}"/>
-      <origin rpy="0 0 0" xyz="0.018 0.00 0.00438"/>
-      <axis xyz="0 0 ${rotor_direction}"/>
-    </joint>
     #### rotor joint (virtual) ####
     <joint name="rotor${self}" type="continuous">
       <limit effort="100.0" lower="${min_force}" upper="${max_force}" velocity="0.5"/>
-      <parent link="rotor_parent${self}"/>
+      <parent link="gimbal_link${self}"/>
       <child link="thrust${self}"/>
-      <origin rpy="0 0 0" xyz="0 0 0"/>
+      <origin rpy="0 0 0" xyz="0.018 0.00 0.00438"/>
       <axis xyz="0 0 ${rotor_direction}"/>
     </joint>
