Commit message: [Beetle][Vision] workaound enabling tag detection.

File: robots/beetle/robots/beetle.gazebo.xacro (robot description, xacro)
@@ -24,3 +24,69 @@
     </plugin>
   </gazebo>
+  <gazebo reference="base_link">
+    <mu1>0.1</mu1>
+    <mu2>0.1</mu2>
+  </gazebo>
+  <!-- sensors -->
+  <!-- 1. stereo camera: depth, color based on left camera -->
+  <xacro:extra_module name = "downward_camera_frame" parent = "base_link">
+    <origin xyz="0.0 0.00 0.0" rpy="0 ${pi/2} 0"/>
+    <inertial>
+      <mass value = "0.00001" />
+      <origin xyz="0 0 0" rpy="0 0 0"/>
+      <inertia
+          ixx="0.000001" ixy="0.0" ixz="0.0"
+          iyy="0.000001" iyz="0.0"
+          izz="0.000002"/>
+    </inertial>
+  </xacro:extra_module>
+  <xacro:extra_module name = "downward_camera_optical_frame" parent = "downward_camera_frame">
+    <origin xyz="0 0 0" rpy="${-pi / 2} 0 ${-pi / 2}"/>
+    <inertial>
+      <mass value = "0.00001" />
+      <origin xyz="0 0 0" rpy="0 0 0"/>
+      <inertia
+          ixx="0.000001" ixy="0.0" ixz="0.0"
+          iyy="0.000001" iyz="0.0"
+          izz="0.000002"/>
+    </inertial>
+  </xacro:extra_module>
+  <!-- gazebo plugin -->
+  <gazebo reference="downward_camera_frame">
+    <sensor type="camera" name="downward_camera">
+      <update_rate>30.0</update_rate>
+      <camera name="head">
+        <horizontal_fov>1.57</horizontal_fov>
+        <image>
+          <width>640</width>
+          <height>480</height>
+          <format>R8G8B8</format>
+        </image>
+        <clip>
+          <near>0.02</near>
+          <far>300</far>
+        </clip>
+        <noise>
+          <type>gaussian</type>
+          <mean>0.0</mean>
+          <stddev>0.007</stddev>
+        </noise>
+      </camera>
+      <plugin name="camera_controller" filename="libgazebo_ros_camera.so">
+        <robotNamespace>$(arg robot_name)</robotNamespace>
+        <alwaysOn>true</alwaysOn>
+        <updateRate>0.0</updateRate>
+        <cameraName>downword_camera</cameraName>
+        <imageTopicName>image_raw</imageTopicName>
+        <cameraInfoTopicName>camera_info</cameraInfoTopicName>
+        <frameName>downward_camera_optical_frame</frameName>
+        <hackBaseline>0.07</hackBaseline>
+        <distortionK1>0.0</distortionK1>
+        <distortionK2>0.0</distortionK2>
+        <distortionK3>0.0</distortionK3>
+        <distortionT1>0.0</distortionT1>
+        <distortionT2>0.0</distortionT2>
+      </plugin>
+    </sensor>
+  </gazebo>
 </robot>

File: robots/beetle/urdf/beetle.urdf.xacro (robot description, xacro)
@@ -198,3 +198,22 @@
     </transmission>
   </xacro:macro>
+  <!--extra module-->
+  <xacro:macro name="extra_module" params="name parent *origin *inertial visible:=0 model_url:=1 scale:=1">
+    <joint name="${parent}2${name}" type="fixed">
+      <parent link="${parent}"/>
+      <child link="${name}"/>
+      <xacro:insert_block name="origin" />
+    </joint>
+    <link name="${name}">
+      <xacro:insert_block name="inertial" />
+      <xacro:if value="${visible == 1}">
+        <visual>
+          <origin rpy="0 0 0" xyz="0 0 0"/>
+          <geometry>
+            <mesh filename="${model_url}" scale= "${scale} ${scale} ${scale}"/>
+          </geometry>
+        </visual>
+      </xacro:if>
+    </link>
+  </xacro:macro>
 </robot>

Commit message: [Beetle][Apriltag] workaround attaching apriltags to beetle airframe.

File: robots/beetle/robots/beetle.gazebo.xacro (robot description, xacro)
@@ -28,8 +28,14 @@
     <mu2>0.1</mu2>
   </gazebo>
+  <gazebo reference="apriltag_1">
+    <material>Apriltag36_11_00000</material>
+  </gazebo>
+  <gazebo reference="apriltag_2">
+    <material>Apriltag36_11_00000</material>
+  </gazebo>
   <!-- sensors -->
   <!-- 1. stereo camera: depth, color based on left camera -->
   <xacro:extra_module name = "downward_camera_frame" parent = "base_link">
-    <origin xyz="0.0 0.00 0.0" rpy="0 ${pi/2} 0"/>
+    <origin xyz="0.24 -0.32 0.18" rpy="0 0 0"/>
     <inertial>
       <mass value = "0.00001" />
@@ -90,3 +96,94 @@
     </sensor>
   </gazebo>
+  <!-- tags -->
+  <joint name="apriltag_joint_1" type="fixed">
+    <parent link="base_link"/>
+    <child link="apriltag_1"/>
+    <origin rpy="0 ${pi/2.0} 0" xyz="0.27 0.33 0.18"/>
+    <axis xyz="0 0 1"/>
+  </joint>
+  <link name="apriltag_1">
+    <inertial>
+      <origin xyz="0 0 0" rpy="0 0 0"/>
+      <mass value="0.00001"/>
+      <inertia
+          ixx="0.000001" ixy="0.0" ixz="0.0"
+          iyy="0.000001" iyz="0.0"
+          izz="0.000001"/>
+    </inertial>
+    <visual>
+      <origin xyz="0 0 0" rpy="0 0 0"/>
+      <geometry>
+  	<box size="0.2 0.2 0.01"/>
+      </geometry>
+      <material name = "Apriltag36_11_00000"/>
+    </visual>
+  </link>
+  <joint name="tag_cover_joint_1" type="fixed">
+    <parent link="apriltag_1"/>
+    <child link="tag_cover_1"/>
+    <origin rpy="0 0 0" xyz="0 0 -0.005"/>
+    <axis xyz="0 0 1"/>
+  </joint>
+  <link name="tag_cover_1">
+    <inertial>
+      <origin xyz="0 0 0" rpy="0 0 0"/>
+      <mass value="0.00001"/>
+      <inertia
+          ixx="0.000001" ixy="0.0" ixz="0.0"
+          iyy="0.000001" iyz="0.0"
+          izz="0.000001"/>
+    </inertial>
+    <visual>
+      <origin xyz="0 0 0" rpy="0 0 0"/>
+      <geometry>
+  	<box size="0.2 0.2 0.01"/>
+      </geometry>
+    </visual>
+  </link>
+  <joint name="apriltag_joint_2" type="fixed">
+    <parent link="base_link"/>
+    <child link="apriltag_2"/>
+    <origin rpy="0 ${pi/2.0} 0" xyz="-0.27 -0.33 0.18"/>
+    <axis xyz="0 0 1"/>
+  </joint>
+  <link name="apriltag_2">
+    <inertial>
+      <origin xyz="0 0 0" rpy="0 0 0"/>
+      <mass value="0.00001"/>
+      <inertia
+          ixx="0.000001" ixy="0.0" ixz="0.0"
+          iyy="0.000001" iyz="0.0"
+          izz="0.000001"/>
+    </inertial>
+    <visual>
+      <origin xyz="0 0 0" rpy="0 0 ${pi}"/>
+      <geometry>
+  	<box size="0.2 0.2 0.01"/>
+      </geometry>
+      <!-- <material name = "Apriltag36_11_00000"/> -->
+    </visual>
+  </link>
+  <joint name="tag_cover_joint_2" type="fixed">
+    <parent link="apriltag_2"/>
+    <child link="tag_cover_2"/>
+    <origin rpy="0 0 0" xyz="0 0 0.005"/>
+    <axis xyz="0 0 1"/>
+  </joint>
+  <link name="tag_cover_2">
+    <inertial>
+      <origin xyz="0 0 0" rpy="0 0 0"/>
+      <mass value="0.00001"/>
+      <inertia
+          ixx="0.000001" ixy="0.0" ixz="0.0"
+          iyy="0.000001" iyz="0.0"
+          izz="0.000001"/>
+    </inertial>
+    <visual>
+      <origin xyz="0 0 0" rpy="0 0 0"/>
+      <geometry>
+  	<box size="0.2 0.2 0.01"/>
+      </geometry>
+    </visual>
+  </link>
 </robot>

Commit message: [Beetle] modified for docking by apriltag.

File: robots/beetle/robots/beetle.gazebo.xacro (robot description, xacro)
@@ -100,5 +100,5 @@
     <parent link="base_link"/>
     <child link="apriltag_1"/>
-    <origin rpy="0 ${pi/2.0} 0" xyz="0.27 0.33 0.18"/>
+    <origin rpy="0 ${pi/2.0} 0" xyz="0.0 0.36 0.18"/>
     <axis xyz="0 0 1"/>
   </joint>
@@ -145,5 +145,5 @@
     <parent link="base_link"/>
     <child link="apriltag_2"/>
-    <origin rpy="0 ${pi/2.0} 0" xyz="-0.27 -0.33 0.18"/>
+    <origin rpy="0 ${pi/2.0} 0" xyz="-0.0 -0.36 0.18"/>
     <axis xyz="0 0 1"/>
   </joint>
