Commit message: [Twin_Hammer][robot_model][urdf] rewrite urdf parameters add mesf files create plugins modefy some configs TODO debug around RobotModel and ControlBase

File: robots/twin_hammer/urdf/device.urdf.xacro (robot description, xacro)
@@ -1,5 +1,5 @@
 <?xml version="1.0"?>
 <robot
-    xmlns:xacro="http://www.ros.org/wiki/xacro" name="twin_hammer" >
+    xmlns:xacro="http://www.ros.org/wiki/xacro" name="Twin_Hammer" >
   <baselink name="fc" />
   <thrust_link name="thrust" />
@@ -8,7 +8,7 @@
   <xacro:property name="rod_length" value="1.0" />
   <xacro:property name="link_length" value=".424" />
-  <xacro:property name="gimbal_roll_x_offset" value="0.2" />
-  <xacro:property name="gimbal_pitch_z_offset" value="0.037" />
-  <xacro:property name="PC_mount_offset" value="0.2" />
+  <xacro:property name="gimbal_roll_x_offset" value="0.0362" />
+  <xacro:property name="gimbal_pitch_x_offset" value="0.0065" />
+  <xacro:property name="gimbal_pitch_z_offset" value="0.0265" />
   <!-- dynamics -->
   <m_f_rate value="0" /> <!-- drug torque rate -->
@@ -28,36 +28,36 @@
   </xacro:macro>
   <!-- gimbal unit with rotor -->
-  <xacro:macro name="gimbal_unit" params="ID"> <!-- ID:1 is spinal side, ID:2 is another side-->
+  <xacro:macro name="gimbal_unit" params="id"> <!-- id:1 is spinal side, id:2 is another side-->
     <!-- gimbal roll -->
-    <joint name="gimbal${ID}_roll" type="revolute">
+    <joint name="gimbal${id}_roll" type="revolute">
       <limit effort="3" lower="-3.14" upper="3.14" velocity="12.5"/>
       <parent link="main_body"/>
-      <child link="gimbal${ID}_roll_module"/>
-      <xacro:if value="${ID == 1}" >
-        <origin rpy="0 0 0" xyz="${gimbal_roll_x_offset} 0 0"/>
-      </xacro:if>
-      <xacro:if value="${ID == 2}" >
-        <origin rpy="0 0 0" xyz="${rod_length - gimbal_roll_x_offset} 0 0"/>
+      <child link="gimbal${id}_roll_module"/>
+      <xacro:if value="${id == 1}" >
+        <origin rpy="0 0 0" xyz="${rod_length*0.5 - gimbal_roll_x_offset} 0 0"/>
+      </xacro:if>
+      <xacro:if value="${id == 2}" >
+        <origin rpy="0 0 0" xyz="${gimbal_roll_x_offset - rod_length*0.5} 0 0"/>
       </xacro:if>
       <axis xyz="1 0 0"/>
       <dynamics damping="0.1" friction="0.0"/>
     </joint>
-    <link name="gimbal${ID}_roll_module">
-      <inertial>
-        <origin xyz="${gimbal_roll_x_offset - 17.60 * 0.001} ${0.42 * 0.001} ${15.48 * 0.001}" rpy="0 0 0"/>
-        <mass value="0.4604" />
-        <inertia
-            ixx="0.0004" iyy="0.0004" izz="0.0003"
-            ixy="0" ixz="-0.0003" iyz="0"/>
+    <link name="gimbal${id}_roll_module">
+      <inertial>
+        <origin xyz="-0.0151 0.0012 0.0233" rpy="0 0 0"/>
+        <mass value="0.3335" />
+        <inertia
+            ixx="0.0008" iyy="0.0009" izz="0.0003"
+            ixy="0" ixz="-0.0002" iyz="0"/>
       </inertial>
       <visual>
-        <xacro:if value="{ID == 1}">
-          <origin xyz="${gimbal_roll_x_offset} 0 0" rpy="0 0 0"/>
-        </xacro:if>
-        <xacro:if value="{ID == 2}">
-          <origin xyz="${rod_length - gimbal_roll_x_offset} 0 0" rpy="0 0 ${pi}"/>
-        </xacro:if>
-        <geometry>
-          <mesh filename="package://dragon/urdf/mesh/ducted_fan_gimbal_roll.dae"/>
+        <xacro:if value="${id == 1}">
+          <origin xyz="0 0 0" rpy="0 0 0"/>
+        </xacro:if>
+        <xacro:if value="${id == 2}">
+          <origin xyz="0 0 0" rpy="0 0 ${pi}"/>
+        </xacro:if>
+        <geometry>
+          <mesh filename="package://twin_hammer/urdf/mesh/gimbal_roll_module.dae" scale="0.001 0.001 0.001"/>
         </geometry>
       </visual>
@@ -66,5 +66,5 @@
         <origin rpy="0 0 0" xyz="${gimbal_roll_x_offset}  0 0"/>
         <geometry>
-          <box size="0.1 0.3 0.1686"/>
+          <box size="0.103 0.064 0.156"/>
         </geometry>
       </collision>
@@ -79,41 +79,46 @@
     </link>
     <!-- gimbal pitch -->
-    <joint name="gimbal${ID}_pitch" type="revolute">
+    <joint name="gimbal${id}_pitch" type="revolute">
       <limit effort="3" lower="-3.14" upper="3.14" velocity="12.5"/>
-      <parent link="gimbal${ID}_roll_module"/>
-      <child link="gimbal${ID}_pitch_module"/>
-      <origin rpy="0 0 0" xyz="0 0 ${gimbal_pitch_z_offset}"/>
+      <parent link="gimbal${id}_roll_module"/>
+      <child link="gimbal${id}_pitch_module"/>
+      <xacro:if value="${id == 1}" >
+        <origin rpy="0 0 0" xyz="${gimbal_pitch_x_offset} 0 ${gimbal_pitch_z_offset}"/>
+      </xacro:if>
+      <xacro:if value="${id == 2}" >
+        <origin rpy="0 0 0" xyz="${-gimbal_pitch_x_offset} 0 ${gimbal_pitch_z_offset}"/>
+      </xacro:if>
       <axis xyz="0 1 0"/>
       <dynamics damping="0.1" friction="0.0"/>
     </joint>
-    <link name="gimbal${ID}_pitch_module">
-      <inertial>
-        <origin xyz="0 ${0.33 * 0.001}  ${-8.71 * 0.001}" rpy="0 0 0"/>
-        <mass value="0.5301" />
-        <inertia
-            ixx="0.0061" iyy="0.0001" izz="0.0061"
+    <link name="gimbal${id}_pitch_module">
+      <inertial>
+        <origin xyz="0 0.0005 -0.0092" rpy="0 0 0"/>
+        <mass value="0.5276" />
+        <inertia
+            ixx="0.0063" iyy="0.0004" izz="0.0062"
             ixy="0.0" ixz="0.0" iyz="0.0"/>
       </inertial>
       <visual>
-        <xacro:if value="${ID == 1}" >
+        <xacro:if value="${id == 1}" >
           <origin xyz="0 0 0" rpy="0 0 0"/>
         </xacro:if>
-        <xacro:if value="${ID == 2}" >
+        <xacro:if value="${id == 2}" >
           <origin xyz="0 0 0" rpy="0 0 ${pi}"/>
         </xacro:if>
         <geometry>
-          <mesh filename="package://dragon/urdf/mesh/ducted_fan_gimbal_pitch.dae"/>
+          <mesh filename="package://twin_hammer/urdf/mesh/gimbal_pitch_module.dae" scale="0.001 0.001 0.001"/>
         </geometry>
       </visual>
     </link>
     <!-- rotor -->
-    <joint name="rotor${ID}" type="continuous">
+    <joint name="rotor${id}" type="continuous">
       <limit effort="100.0" lower="${min_force}" upper="${max_force}" velocity="0.5"/>
-      <parent link="gimbal${ID}_pitch_module"/>
-      <child link="thrust${ID}"/>
+      <parent link="gimbal${id}_pitch_module"/>
+      <child link="thrust${id}"/>
       <origin rpy="0 0 0" xyz="0 0 0"/>
       <axis xyz="0 0 1"/>
     </joint>
-    <link name="thrust${ID}">
+    <link name="thrust${id}">
       <inertial>
         <origin xyz="0 0 0" rpy="0 0 0"/>
@@ -126,11 +131,11 @@
     </link>
     <!-- special part of duct fun -->
-    <joint name="edf${ID}_left_mount" type="fixed">
-      <child link="edf${ID}_left"/>
-      <parent link="gimbal${ID}_pitch_module"/>
+    <joint name="edf${id}_left_mount" type="fixed">
+      <child link="edf${id}_left"/>
+      <parent link="gimbal${id}_pitch_module"/>
       <origin rpy="0 0 0" xyz="0 0.1115 0 "/>
       <axis xyz="0 0 1"/>
     </joint>
-    <link name="edf${ID}_left">
+    <link name="edf${id}_left">
       <inertial>
         <origin xyz="0 0 0" rpy="0 0 0"/>
@@ -142,11 +147,11 @@
       </inertial>
     </link>
-    <joint name="edf${ID}_right_mount" type="fixed">
-      <child link="edf${ID}_right"/>
-      <parent link="gimbal${ID}_pitch_module"/>
+    <joint name="edf${id}_right_mount" type="fixed">
+      <child link="edf${id}_right"/>
+      <parent link="gimbal${id}_pitch_module"/>
       <origin rpy="0 0 0" xyz="0 -0.1115 0 "/>
       <axis xyz="0 0 1"/>
     </joint>
-    <link name="edf${ID}_right">
+    <link name="edf${id}_right">
       <inertial>
         <origin xyz="0 0 0" rpy="0 0 0"/>
@@ -158,32 +163,32 @@
       </inertial>
     </link>
-    <xacro:damping_factor link ="thrust${ID}"/>
+    <xacro:damping_factor link ="thrust${id}"/>
     <!-- hardware interface -->
-    <transmission name="gimbal${ID}_roll_tran">
+    <transmission name="gimbal${id}_roll_tran">
       <type>transmission_interface/SimpleTransmission</type>
-      <joint name="gimbal${ID}_roll">
+      <joint name="gimbal${id}_roll">
         <hardwareInterface>hardware_interface/EffortJointInterface</hardwareInterface>
       </joint>
-      <actuator name="gimbal_servo{ID}_roll">
+      <actuator name="gimbal_servo{id}_roll">
         <hardwareInterface>hardware_interface/EffortJointInterface</hardwareInterface>
         <mechanicalReduction>1</mechanicalReduction>
       </actuator>
     </transmission>
-    <transmission name="gimbal${ID}_pitch_tran">
+    <transmission name="gimbal${id}_pitch_tran">
       <type>transmission_interface/SimpleTransmission</type>
-      <joint name="gimbal${ID}_pitch">
+      <joint name="gimbal${id}_pitch">
         <hardwareInterface>hardware_interface/EffortJointInterface</hardwareInterface>
       </joint>
-      <actuator name="gimbal_servo{ID}_pitch">
+      <actuator name="gimbal_servo{id}_pitch">
         <hardwareInterface>hardware_interface/EffortJointInterface</hardwareInterface>
         <mechanicalReduction>1</mechanicalReduction>
       </actuator>
     </transmission>
-    <transmission name="rotor${ID}_tran">
+    <transmission name="rotor${id}_tran">
       <type>transmission_interface/SimpleTransmission</type>
-      <joint name="rotor${ID}">
+      <joint name="rotor${id}">
         <hardwareInterface>RotorInterface</hardwareInterface>
       </joint>
-      <actuator name="rotor${ID}">
+      <actuator name="rotor${id}">
         <hardwareInterface>RotorInterface</hardwareInterface>
         <mechanicalReduction>1</mechanicalReduction>
@@ -212,15 +217,15 @@
   <link name="main_body">
     <inertial>
-      <mass value = "0.432" />
-      <origin xyz="${rod_length} 0 0.017" rpy="0 0 0"/>
+      <mass value = "0.25" />
+      <origin xyz="-0.0001 -0.0139 0.1356" rpy="0 0 0"/>
       <inertia
-          ixx="0.0021" ixy="0" ixz="0"
-          iyy="0.0015" iyz="0"
-          izz="0.0032"/>
+          ixx="0.0175" ixy="0" ixz="0"
+          iyy="0.0174" iyz="-0.0007"
+          izz="0.0002"/>
     </inertial>
     <visual>
-      <origin rpy="0 0 0" xyz="0 0 0"/>
+      <origin rpy="${pi/2} 0 ${pi/2}" xyz="-0.8 0 0"/>
       <geometry>
-        <mesh filename="package://mini_quadrotor/urdf/mesh/main_body.dae" />
+        <mesh filename="package://twin_hammer/urdf/mesh/main_body.dae" scale="0.001 0.001 0.001"/>
       </geometry>
     </visual>
@@ -247,8 +252,8 @@
     <child link="fc"/>
     <parent link="main_body"/>
-    <origin rpy="0 0 0" xyz="0.316 -0.004 0.043"/>
+    <origin rpy="0 0 0" xyz="0.2341 0 0.0292"/>
     <axis xyz="0 0 1"/>
   </joint>
-  <xacro:gimbal_unit ID = "1" />
-  <xacro:gimbal_unit ID = "2" />
+  <xacro:gimbal_unit id="1" />
+  <xacro:gimbal_unit id="2" />
 </robot>
