Commit message: [Twin Hammer] [urdf] [gazebo] tried to apply ft_sensor plugin it hasnt completed gave up

File: robots/twin_hammer/urdf/device.gazebo.xacro (robot description, xacro)
@@ -12,3 +12,12 @@
     <mu2>0.1</mu2>
   </gazebo>
+  <!-- <gazebo reference="root_to_dummyweight_joint">
+    <plugin name="force_torque_plugin" filename="libgazebo_ros_ft_sensor.so">
+      <always_on>true</always_on>
+      <update_rate>100.0</update_rate>
+      <sensor_type>force_torque</sensor_type>
+      <jointName>root_to_dummyweight_joint</jointName>
+      <topicName>/twin_hammer/ftsensor_gazebo</topicName>
+    </plugin>
+  </gazebo> -->
 </robot>

File: robots/twin_hammer/urdf/device.urdf.xacro (robot description, xacro)
@@ -1,5 +1,5 @@
 <?xml version="1.0"?>
 <robot
-   xmlns:xacro="http://www.ros.org/wiki/xacro" name="Twin_Hammer" >
+   xmlns:xacro="http://www.ros.org/wiki/xacro" name="twin_hammer" >
  <baselink name="fc" />
  <thrust_link name="thrust" />
@@ -26,4 +26,20 @@
      <dampingFactor>0.00</dampingFactor>
    </gazebo>
+ </xacro:macro>
+ <!-- ft_sensor -->
+ <xacro:macro name="add_ft_sensor" params="joint_name sensor_topic_name">
+  <gazebo reference="${joint_name}">
+    <sensor type="force_torque" name="${joint_name}_sensor">
+      <always_on>true</always_on>
+      <update_rate>100.0</update_rate>
+      <joint_name>${joint_name}</joint_name>
+      <plugin name="${joint_name}_gazebo_ros_ft_sensor" filename="libgazebo_ros_force_torque.so">
+        <ros>
+          <namespace>/twin_hammer</namespace>
+          <remapping>sensor_data:=${sensor_topic_name}</remapping>
+        </ros>
+      </plugin>
+    </sensor>
+  </gazebo>
  </xacro:macro>
  <!-- <xacro:macro name="rotor" params="number"> -->
@@ -265,4 +281,11 @@
     <origin rpy="0 0 0" xyz="0 0 1.0"/>
   </joint>
+  <!-- ft_sensor_gazebo joint -->
+  <!-- <joint name="root_to_dummyweight_joint" type="fixed">
+    <parent link="dummy_weight"/>
+    <child link="root"/>
+    <origin xyz="0 0 1.0" rpy="0 0 0"/>
+    <xacro:add_ft_sensor joint_name="root_to_dummyweight_joint" sensor_topic_name="/gazebo_ft_sensor"/>
+  </joint> -->
  <!-- main_body -->
  <link name="main_body">
