Commit message: Revert "[Twin_Hammer]"
This reverts commit bffeedc2d62df8ca7971e01ad00eca18bcd701c4.

File: robots/mini_quadrotor/urdf/robot.urdf.xacro (robot description, xacro)
@@ -6,6 +6,6 @@
   <thrust_link name="thrust" />
   <!-- kinematics [m] -->
-  <xacro:property name="rotor_x" value="0.085" />
-  <xacro:property name="rotor_y" value="0.085" />
+  <xacro:property name="rotor_x" value="0.070" />
+  <xacro:property name="rotor_y" value="0.086" />
   <xacro:property name="rotor_z" value="0.026" />
   <!-- dynamics -->
@@ -96,15 +96,15 @@
   <link name="main_body">
     <inertial>
-      <mass value = "0.832" />
-      <origin xyz="0.002 0 ${0.028 - 0.002}" rpy="0 0 0"/> <!-- TODO: true cog pos -->
+      <mass value = "0.432" />
+      <origin xyz="0 0 0.017" rpy="0 0 0"/>
       <inertia
-          ixx="0.0030" ixy="0" ixz="0"
-          iyy="0.0030" iyz="0"
-          izz="0.0045"/>
+          ixx="0.0021" ixy="0" ixz="0"
+          iyy="0.0015" iyz="0"
+          izz="0.0032"/>
     </inertial>
     <visual>
       <origin rpy="0 0 0" xyz="0 0 0"/>
       <geometry>
-        <mesh filename="package://mini_quadrotor/urdf/mesh/main_body_livox.dae" />
+        <mesh filename="package://mini_quadrotor/urdf/mesh/main_body.dae" />
       </geometry>
     </visual>
@@ -127,18 +127,7 @@
     </inertial>
   </xacro:extra_module>
-  <!-- livox mid360 -->
-  <xacro:extra_module name = "lidar_imu" parent = "main_body" visible = "0" > <!-- should be IMU frame -->
-    <origin xyz="${0.011} ${0.02329} ${0.0425 + 0.047 - 0.04412}" rpy="0 0 0"/> <!-- TODO: the true pos -->
-    <inertial>
-      <mass value = "00" />
-      <origin xyz="0 0 0" rpy="0 0 0"/>
-      <inertia
-          ixx="0.0" ixy="0.0" ixz="0.0"
-          iyy="0.0" iyz="0.0" izz="0.0"/>
-    </inertial>
-  </xacro:extra_module>
   <!-- battery -->
   <xacro:extra_module name = "battery" parent = "main_body" visible = "1" model_url = "package://mini_quadrotor/urdf/mesh/turnigy_3S_2200mAh.dae" >
-    <origin xyz="0.0 0 -0.035" rpy="${pi/2} 0 0"/>
+    <origin xyz="0.0105 0 -0.012" rpy="0 0 0"/>
     <inertial>
       <mass value = "0.188" />
