Commit message: [Ninja] Add selectable CFS model and correct wrench estimation

File: robots/ninja/robots/ninja.urdf.xacro (robot description, xacro)
@@ -2,4 +2,8 @@
 <robot
     xmlns:xacro="http://www.ros.org/wiki/xacro" name="ninja" >
+  <!-- Keep the normal-flight model as the default.  The wrench-sensor model
+       restores the dock geometry and inertial parameters used by the CFS
+       experiment before commit 434793c5. -->
+  <xacro:arg name="wrench_sensor" default="false" />
   <xacro:include filename="$(find ninja)/urdf/ninja.urdf.xacro" />
   <xacro:include filename="$(find ninja)/urdf/common.xacro" />
@@ -8,6 +12,6 @@
   <xacro:ninja_gimbal_link self="2" rotor_direction="-1"/>
   <xacro:ninja_gimbal_link self="3" rotor_direction="1"/>
-  <xacro:ninja_docking_mech_yaw/>
-  <xacro:ninja_docking_mech_pitch/>
+  <xacro:ninja_docking_mech_yaw wrench_sensor="$(arg wrench_sensor)"/>
+  <xacro:ninja_docking_mech_pitch wrench_sensor="$(arg wrench_sensor)"/>
   <!-- <xacro:battery_3000mAh/> -->
   <xacro:battery_1300mAh/>

File: robots/ninja/urdf/ninja.urdf.xacro (robot description, xacro)
@@ -111,20 +111,38 @@
    <xacro:friction self="main_body"/>
   </xacro:macro>
-  <xacro:macro name="ninja_docking_mech_yaw">
+  <xacro:macro name="ninja_docking_mech_yaw" params="wrench_sensor:=false">
     <!-- yaw -->
     <link name="yaw_dock_link">
       <inertial>
-        <origin xyz="0.07707992 0.00034225 -0.02807178" rpy="0 0 0"/>
-        <mass value="0.33699537"/>
-        <inertia
-            ixx = "0.00047120" ixy = "-0.00000696" ixz = "-0.00002605"
-            iyx = "-0.00000696" iyy = "0.00089048" iyz = "0.00000963"
-            izx = "-0.00002605" izy = "0.00000963" izz = "0.00082655"/>
-      </inertial>
-      <visual>
-        <origin xyz="0 0 0" rpy="0 0 0"/>
-       <geometry>
-          <mesh filename="package://ninja/urdf/mesh/male_dock_mech.dae" scale="1 1 1"/>
-        </geometry>
+        <xacro:if value="${wrench_sensor}">
+          <origin xyz="0.06461625 0.00000000 -0.02429533" rpy="0 0 0"/>
+          <mass value="0.45686952"/>
+          <inertia
+              ixx = "0.00058684" ixy = "-0.00000696" ixz = "-0.00002605"
+              iyx = "-0.00000696" iyy = "0.00234155" iyz = "0.00000963"
+              izx = "-0.00002605" izy = "0.00000963" izz = "0.00267053"/>
+        </xacro:if>
+        <xacro:unless value="${wrench_sensor}">
+          <origin xyz="0.07707992 0.00034225 -0.02807178" rpy="0 0 0"/>
+          <mass value="0.33699537"/>
+          <inertia
+              ixx = "0.00047120" ixy = "-0.00000696" ixz = "-0.00002605"
+              iyx = "-0.00000696" iyy = "0.00089048" iyz = "0.00000963"
+              izx = "-0.00002605" izy = "0.00000963" izz = "0.00082655"/>
+        </xacro:unless>
+      </inertial>
+      <visual>
+        <xacro:if value="${wrench_sensor}">
+          <origin xyz="0 0 0" rpy="${pi/2} 0 0"/>
+          <geometry>
+            <mesh filename="package://ninja/urdf/mesh/male_dock_module_wrench_test.STL" scale="1 1 1"/>
+          </geometry>
+        </xacro:if>
+        <xacro:unless value="${wrench_sensor}">
+          <origin xyz="0 0 0" rpy="0 0 0"/>
+          <geometry>
+            <mesh filename="package://ninja/urdf/mesh/male_dock_mech.dae" scale="1 1 1"/>
+          </geometry>
+        </xacro:unless>
       </visual>
       <collision>
@@ -167,5 +185,10 @@
       <parent link="yaw_dock_link"/>
       <child link="yaw_connect_point"/>
-      <origin rpy="0 0 0" xyz="0.14085 0 -0.030"/>
+      <xacro:if value="${wrench_sensor}">
+        <origin rpy="0 0 0" xyz="0.0965 0 -0.025"/>
+      </xacro:if>
+      <xacro:unless value="${wrench_sensor}">
+        <origin rpy="0 0 0" xyz="0.14085 0 -0.030"/>
+      </xacro:unless>
       <axis xyz="0 0 1"/>
     </joint>
@@ -234,4 +257,7 @@
       <origin rpy="0 0 0" xyz="0.162845 0.09285 0"/>
       <axis xyz="0 1 0"/>
+      <xacro:if value="$(arg wrench_sensor)">
+        <dynamics damping="0.8" friction="0.0"/>
+      </xacro:if>
     </joint>
     <transmission name="joint_tran${2*self}">
@@ -307,20 +333,37 @@
     </transmission>
   </xacro:macro>
-  <xacro:macro name="ninja_docking_mech_pitch">
+  <xacro:macro name="ninja_docking_mech_pitch" params="wrench_sensor:=false">
     <!-- pitch -->
     <link name="pitch_dock_link">
       <inertial>
-        <origin xyz="-0.04795875 0.02306659 0.00003088" rpy="0 0 0"/>
-        <mass value="0.17183088"/>
-        <inertia
-            ixx = "0.00035938" ixy = "-0.00001594" ixz = "0.00000012"
-            iyx = "-0.00001594" iyy = "0.00038919" iyz = "0.00006568"
-            izx = "0.00000012" izy = "0.00006568" izz = "0.00032884"/>
+        <xacro:if value="${wrench_sensor}">
+          <origin xyz="-0.03575946 0.02293296 0.0000" rpy="0 0 0"/>
+          <mass value="0.16575426"/>
+          <inertia
+              ixx = "0.00023487" ixy = "-0.00014777" ixz = "0.00000012"
+              iyx = "-0.00014777" iyy = "0.00033710" iyz = "0.00000000"
+              izx = "0.00000012" izy = "0.00006568" izz = "0.00044705"/>
+        </xacro:if>
+        <xacro:unless value="${wrench_sensor}">
+          <origin xyz="-0.04795875 0.02306659 0.00003088" rpy="0 0 0"/>
+          <mass value="0.17183088"/>
+          <inertia
+              ixx = "0.00035938" ixy = "-0.00001594" ixz = "0.00000012"
+              iyx = "-0.00001594" iyy = "0.00038919" iyz = "0.00006568"
+              izx = "0.00000012" izy = "0.00006568" izz = "0.00032884"/>
+        </xacro:unless>
       </inertial>
       <visual>
         <origin xyz="0 0 0" rpy="${pi} ${pi} 0"/>
-        <geometry>
-          <mesh filename="package://ninja/urdf/mesh/female_dock_mech.dae" scale="1 1 1"/>
-        </geometry>
+        <xacro:if value="${wrench_sensor}">
+          <geometry>
+            <mesh filename="package://ninja/urdf/mesh/female_dock_module_wrench_test.STL" scale="1 1 1"/>
+          </geometry>
+        </xacro:if>
+        <xacro:unless value="${wrench_sensor}">
+          <geometry>
+            <mesh filename="package://ninja/urdf/mesh/female_dock_mech.dae" scale="1 1 1"/>
+          </geometry>
+        </xacro:unless>
       </visual>
       <collision>
@@ -363,5 +406,10 @@
       <parent link="pitch_dock_link"/>
       <child link="pitch_connect_point"/>
-      <origin rpy="0 0 0" xyz="-0.037 0.025 0"/>
+      <xacro:if value="${wrench_sensor}">
+        <origin rpy="0 0 0" xyz="-0.0645 0.025 0"/>
+      </xacro:if>
+      <xacro:unless value="${wrench_sensor}">
+        <origin rpy="0 0 0" xyz="-0.037 0.025 0"/>
+      </xacro:unless>
       <axis xyz="0 0 1"/>
     </joint>
