Commit message: [Ninja][Mujoco] Add single and two-module flight simulation.

File: robots/ninja/urdf/ninja.urdf.xacro (robot description, xacro)
@@ -234,4 +234,5 @@
       <origin rpy="0 0 0" xyz="0.162845 0.09285 0"/>
       <axis xyz="0 1 0"/>
+      <dynamics damping="0.8" friction="0.0"/>
     </joint>
     <transmission name="joint_tran${2*self}">

Commit message: [Ninja][model] Add models for wrench test

File: robots/ninja/urdf/ninja.urdf.xacro (robot description, xacro)
@@ -115,15 +115,15 @@
     <link name="yaw_dock_link">
       <inertial>
-        <origin xyz="0.07707992 0.00034225 -0.02807178" rpy="0 0 0"/>
-        <mass value="0.33699537"/>
-        <inertia
-            ixx = "0.00047120" ixy = "-0.00000696" ixz = "-0.00002605"
-            iyx = "-0.00000696" iyy = "0.00089048" iyz = "0.00000963"
-            izx = "-0.00002605" izy = "0.00000963" izz = "0.00082655"/>
-      </inertial>
-      <visual>
-        <origin xyz="0 0 0" rpy="0 0 0"/>
+        <origin xyz="0.06461625 -0.02429533 0.00000000" rpy="0 0 0"/>
+        <mass value="0.45686952"/>
+        <inertia
+            ixx = "0.00058684" ixy = "-0.00000696" ixz = "-0.00002605"
+            iyx = "-0.00000696" iyy = "0.00234155" iyz = "0.00000963"
+            izx = "-0.00002605" izy = "0.00000963" izz = "0.00267053"/>
+      </inertial>
+      <visual>
+        <origin xyz="0 0 0" rpy="${pi/2} 0 0"/>
        <geometry>
-          <mesh filename="package://ninja/urdf/mesh/male_dock_mech.dae" scale="1 1 1"/>
+          <mesh filename="package://ninja/urdf/mesh/male_dock_module_wrench_test.STL" scale="1 1 1"/>
         </geometry>
       </visual>
@@ -167,5 +167,5 @@
       <parent link="yaw_dock_link"/>
       <child link="yaw_connect_point"/>
-      <origin rpy="0 0 0" xyz="0.14085 0 -0.030"/>
+      <origin rpy="0 0 0" xyz="0.0965 0 -0.025"/>
       <axis xyz="0 0 1"/>
     </joint>
@@ -312,15 +312,15 @@
     <link name="pitch_dock_link">
       <inertial>
-        <origin xyz="-0.04795875 0.02306659 0.00003088" rpy="0 0 0"/>
-        <mass value="0.17183088"/>
-        <inertia
-            ixx = "0.00035938" ixy = "-0.00001594" ixz = "0.00000012"
-            iyx = "-0.00001594" iyy = "0.00038919" iyz = "0.00006568"
-            izx = "0.00000012" izy = "0.00006568" izz = "0.00032884"/>
+        <origin xyz="-0.03575946 0.02293296 0.0000" rpy="0 0 0"/>
+        <mass value="0.16575426"/>
+        <inertia
+            ixx = "0.00023487" ixy = "-0.00014777" ixz = "0.00000012"
+            iyx = "-0.00014777" iyy = "0.00033710" iyz = "0.00000000"
+            izx = "0.00000012" izy = "0.00006568" izz = "0.00044705"/>
       </inertial>
       <visual>
         <origin xyz="0 0 0" rpy="${pi} ${pi} 0"/>
         <geometry>
-          <mesh filename="package://ninja/urdf/mesh/female_dock_mech.dae" scale="1 1 1"/>
+          <mesh filename="package://ninja/urdf/mesh/female_dock_module_wrench_test.STL" scale="1 1 1"/>
         </geometry>
       </visual>
@@ -364,5 +364,5 @@
       <parent link="pitch_dock_link"/>
       <child link="pitch_connect_point"/>
-      <origin rpy="0 0 0" xyz="-0.037 0.025 0"/>
+      <origin rpy="0 0 0" xyz="-0.0645 0.025 0"/>
       <axis xyz="0 0 1"/>
     </joint>

Commit message: [Ninja][URDF] Fixed the CoG position of dock mech

File: robots/ninja/urdf/ninja.urdf.xacro (robot description, xacro)
@@ -115,5 +115,5 @@
     <link name="yaw_dock_link">
       <inertial>
-        <origin xyz="0.06461625 -0.02429533 0.00000000" rpy="0 0 0"/>
+        <origin xyz="0.06461625 0.00000000 -0.02429533 " rpy="0 0 0"/>
         <mass value="0.45686952"/>
         <inertia

Commit message: [Ninja][Model] revert urdf to normal flight

File: robots/ninja/urdf/ninja.urdf.xacro (robot description, xacro)
@@ -115,15 +115,15 @@
     <link name="yaw_dock_link">
       <inertial>
-        <origin xyz="0.06461625 0.00000000 -0.02429533 " rpy="0 0 0"/>
-        <mass value="0.45686952"/>
-        <inertia
-            ixx = "0.00058684" ixy = "-0.00000696" ixz = "-0.00002605"
-            iyx = "-0.00000696" iyy = "0.00234155" iyz = "0.00000963"
-            izx = "-0.00002605" izy = "0.00000963" izz = "0.00267053"/>
-      </inertial>
-      <visual>
-        <origin xyz="0 0 0" rpy="${pi/2} 0 0"/>
+        <origin xyz="0.07707992 0.00034225 -0.02807178" rpy="0 0 0"/>
+        <mass value="0.33699537"/>
+        <inertia
+            ixx = "0.00047120" ixy = "-0.00000696" ixz = "-0.00002605"
+            iyx = "-0.00000696" iyy = "0.00089048" iyz = "0.00000963"
+            izx = "-0.00002605" izy = "0.00000963" izz = "0.00082655"/>
+      </inertial>
+      <visual>
+        <origin xyz="0 0 0" rpy="0 0 0"/>
        <geometry>
-          <mesh filename="package://ninja/urdf/mesh/male_dock_module_wrench_test.STL" scale="1 1 1"/>
+          <mesh filename="package://ninja/urdf/mesh/male_dock_mech.dae" scale="1 1 1"/>
         </geometry>
       </visual>
@@ -167,5 +167,5 @@
       <parent link="yaw_dock_link"/>
       <child link="yaw_connect_point"/>
-      <origin rpy="0 0 0" xyz="0.0965 0 -0.025"/>
+      <origin rpy="0 0 0" xyz="0.14085 0 -0.030"/>
       <axis xyz="0 0 1"/>
     </joint>
@@ -234,5 +234,4 @@
       <origin rpy="0 0 0" xyz="0.162845 0.09285 0"/>
       <axis xyz="0 1 0"/>
-      <dynamics damping="0.8" friction="0.0"/>
     </joint>
     <transmission name="joint_tran${2*self}">
@@ -312,15 +311,15 @@
     <link name="pitch_dock_link">
       <inertial>
-        <origin xyz="-0.03575946 0.02293296 0.0000" rpy="0 0 0"/>
-        <mass value="0.16575426"/>
-        <inertia
-            ixx = "0.00023487" ixy = "-0.00014777" ixz = "0.00000012"
-            iyx = "-0.00014777" iyy = "0.00033710" iyz = "0.00000000"
-            izx = "0.00000012" izy = "0.00006568" izz = "0.00044705"/>
+        <origin xyz="-0.04795875 0.02306659 0.00003088" rpy="0 0 0"/>
+        <mass value="0.17183088"/>
+        <inertia
+            ixx = "0.00035938" ixy = "-0.00001594" ixz = "0.00000012"
+            iyx = "-0.00001594" iyy = "0.00038919" iyz = "0.00006568"
+            izx = "0.00000012" izy = "0.00006568" izz = "0.00032884"/>
       </inertial>
       <visual>
         <origin xyz="0 0 0" rpy="${pi} ${pi} 0"/>
         <geometry>
-          <mesh filename="package://ninja/urdf/mesh/female_dock_module_wrench_test.STL" scale="1 1 1"/>
+          <mesh filename="package://ninja/urdf/mesh/female_dock_mech.dae" scale="1 1 1"/>
         </geometry>
       </visual>
@@ -364,5 +363,5 @@
       <parent link="pitch_dock_link"/>
       <child link="pitch_connect_point"/>
-      <origin rpy="0 0 0" xyz="-0.0645 0.025 0"/>
+      <origin rpy="0 0 0" xyz="-0.037 0.025 0"/>
       <axis xyz="0 0 1"/>
     </joint>

Commit message: [Ninja][URDF] Corrected mass value of wrench dock mech

File: robots/ninja/urdf/ninja.urdf.xacro (robot description, xacro)
@@ -117,5 +117,5 @@
         <xacro:if value="${wrench_sensor}">
           <origin xyz="0.06461625 0.00000000 -0.02429533" rpy="0 0 0"/>
-          <mass value="0.45686952"/>
+          <mass value="0.38640665"/>
           <inertia
               ixx = "0.00058684" ixy = "-0.00000696" ixz = "-0.00002605"
@@ -339,5 +339,5 @@
         <xacro:if value="${wrench_sensor}">
           <origin xyz="-0.03575946 0.02293296 0.0000" rpy="0 0 0"/>
-          <mass value="0.16575426"/>
+          <mass value="0.09529127"/>
           <inertia
               ixx = "0.00023487" ixy = "-0.00014777" ixz = "0.00000012"
